File: EInkDisplay-PCB/ECE477-SeniorDesign/PowerSheet.kicad_sch (KiCad schematic)
At the start: 9 parts, among them Q2 BSS138

Commit message: Adding Component Library
-named einkcomponent library
Parts:
- removed C3, C4: C, symbol Device:C
- removed D4, D5, D6: MBR0530, Diode_SMD:D_SOD-123, symbol Diode:MBR0530
- removed L2: L, symbol Device:L
- removed Q2: BSS138, Package_TO_SOT_SMD:SOT-23, symbol Transistor_FET:BSS138
- removed R3, R4: R, symbol Device:R
