File: EInkDisplay-PCB/ECE477-SeniorDesign/_autosave-ECE477-SeniorDesign.kicad_pcb (KiCad board)
At the start: 2 copper layers, 69 parts, among them J2 USB_B, J3 JST Conn, J4 JST Conn, J5 JST Conn, J6 Battery Connector, J9 Micro_SD_Card_Det1, U1 CP2102-GMR, U2 MCP73871, U3 STM32L496ZGTxP, U4 TPS63060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

Commit message: power & power pcb layout
Parts:
- added ?: , , F.Cu at (161.9, 121.4)
- added ?: , , F.Cu at (161.2, 125.7)
- added ?: , , F.Cu at (162.2, 125.7)
- added ?: , , F.Cu at (160.7, 126.4)
- added ?: , , F.Cu at (160.2, 125.7)
- added ?: , , F.Cu at (162.4, 119.7)
- added ?: , , F.Cu at (161.4, 119.7)
- added ?: , , F.Cu at (161.9, 120.4)
- added ?: , , F.Cu at (161.7, 126.4)
- added ?: , , F.Cu at (160.9, 121.4)
- added ?: , , F.Cu at (154.8, 119.5)
- added ?: , , F.Cu at (160.9, 120.4)
- added ?: , , F.Cu at (160.4, 119.7)
- added ?: , , F.Cu at (155.5, 119.5)
- added J1: SD_Card_Device, PCB_Lib:SD_Reader, F.Cu at (89.0, 68.2)
- added R2: 20k, Resistor_SMD:R_0805_2012Metric_Pad1.20x1.40mm_HandSolder, F.Cu at (112.1, 62.7)
- added R3: 20k, Resistor_SMD:R_0805_2012Metric_Pad1.20x1.40mm_HandSolder, F.Cu at (112.1, 65.7)
- added R4: 20k, Resistor_SMD:R_0805_2012Metric_Pad1.20x1.40mm_HandSolder, F.Cu at (112.1, 68.6)
- added R5: 20k, Resistor_SMD:R_0805_2012Metric_Pad1.20x1.40mm_HandSolder, F.Cu at (112.1, 71.6)
- added R6: 20k, Resistor_SMD:R_0805_2012Metric_Pad1.20x1.40mm_HandSolder, F.Cu at (112.1, 74.5)
- added R7: 200, Resistor_SMD:R_0805_2012Metric_Pad1.20x1.40mm_HandSolder, F.Cu at (116.8, 62.7)
- added R8: 20k, Resistor_SMD:R_0805_2012Metric_Pad1.20x1.40mm_HandSolder, F.Cu at (116.8, 65.7)
- added R9: 20k, Resistor_SMD:R_0805_2012Metric_Pad1.20x1.40mm_HandSolder, F.Cu at (116.8, 68.6)
- added U9: 74LVC125APW_118, PCB_Lib:74LVC, F.Cu at (16.1, 22.4)
- C33: value C_Small -> 4.7 uF
- C36: value C_Small -> 0.47uF
- L1: footprint Inductor_SMD:L_0805_2012Metric_Pad1.15x1.40mm_HandSolder -> Inductor_SMD:L_1008_2520Metric_Pad1.43x2.20mm_HandSolder
- moved J9 102.4 mm to (8.95, 10.3), turned to 0 degrees
- moved U8 91.3 mm to (6.42, 23.2)
- moved U2 48.9 mm to (122.6, 109.1)
- moved C32 40.0 mm to (164.5, 126.5), turned to 0 degrees
- moved L1 39.9 mm to (161.3, 117.9), turned to 0 degrees
- moved C34 39.2 mm to (169.2, 126.7)
- moved C36 35.9 mm to (177.8, 117.8), turned to -90 degrees
- moved C30 34.0 mm to (155.2, 121.0)
- moved C31 33.4 mm to (157.5, 121.0)
- moved C35 30.0 mm to (165.2, 120.8), turned to -90 degrees
- moved U4 30.0 mm to (161.5, 123.2)
- moved C37 27.4 mm to (167.5, 120.8), turned to -90 degrees
- moved C38 26.9 mm to (169.8, 120.8), turned to -90 degrees
- moved U5 25.9 mm to (182.6, 115.5)
- moved R18 24.8 mm to (118.8, 111.8), turned to -90 degrees
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Connections:
- net /MCU/SPI2_SCK renamed /ExtraPeriphs/SD_SCK
- U3 pad 100: /MCU/SD_GPIO -> unconnected-(U3-PA8-Pad100)
- U3 pad 139: /MCU/SPI2_NSS -> /ExtraPeriphs/SD_CS
- U3 pad 75: /MCU/SPI2_MISO -> /ExtraPeriphs/SD_MISO
- U3 pad 76: /MCU/SPI2_MOSI -> /ExtraPeriphs/SD_MOSI
Routing:
- net +3.3V: track 0.00 -> 7.18 mm
- net Net-(U4-L2): track 0.00 -> 6.88 mm
- net Net-(U4-L1): track 0.00 -> 6.60 mm
- net V_5V: track 0.00 -> 5.96 mm
- net Net-(U4-VAUX): track 0.00 -> 2.34 mm
