File: EInkDisplay-PCB/ECE477-SeniorDesign/LiPoPower_Module_Sheet.kicad_sch (KiCad schematic)
At the start: 0 parts

Commit message: introducing power sch
Parts:
- added C30, C31: 10 uF, symbol Device:C_Small
- added C32: 0.1 uF, symbol Device:C_Small
- added C33, C35: C_Small, symbol Device:C_Small
- added C34: 10 pF, symbol Device:C_Small
- added L1: 1 uH, symbol Device:L
- added R16: 10KΩ, symbol Device:R_Small_US
- added R17, R18: 15KΩ, symbol Device:R_Small_US
- added R19: 1.2 M, symbol Device:R_Small_US
- added R20: 200 K, symbol Device:R_Small_US
- added R21: 10 K, symbol Device:R_Small_US
- added R22: 10 mΩ, symbol Device:R_Small_US
- added U2: MCP73871, Package_DFN_QFN:QFN-20-1EP_4x4mm_P0.5mm_EP2.5x2.5mm, symbol Battery_Management:MCP73871
- added U4: TPS63060, Package_SON:Texas_S-PWSON-N10_ThermalVias, symbol Regulator_Switching:TPS63060
- added U5: BQ27441-G1, Package_SON:Texas_S-PDSO-N12, symbol Battery_Management:BQ27441-G1
Connections:
- new net: L1.1, U4.1 (L1)
- new net: L1.2, U4.10 (L2)
- new net: C32.1, U4.6 (VAUX)
- new net: C34.1, R19.2, R20.1, U4.8 (FB)
- new net: R17.1, U2.12 (PROG3)
- new net: R22.2, U5.7 (SRN)
- new net: C35.1, U5.3 (V_{SS})
- new net: R16.1, U2.13 (PROG1)
- new net: R18.1, U2.5 (THERM)
- new net: R21.2, U5.10 (BIN)
- new net GND: C30.2, C31.2, C32.2, C33.2, C34.2, C35.2, R16.2, R17.2, R18.2, R20.2, R21.1, U2.10 (V_{SS}), U2.11 (V_{SS}), U2.21 (V_{SS}), U2.3 (SEL), U4.11 (PGND), U4.4 (PS/SYNC), U4.7 (GND), U5.5 (V_{DD})
- new net USB_5V: U2.17 (CE), U2.9 (~{TE})
- new net VBAT: R22.1, U2.14 (V_{BAT}), U2.15 (V_{BAT}), U2.16 (V_{BAT_SENSE}), U5.6 (BAT), U5.8 (SRP)
- new net VBUS: U2.18 (IN), U2.19 (IN), U2.2 (VPCC)
- new net V_3.3: R19.1, U4.9 (VOUT)
- new net V_SYS: C30.1, C31.1, C33.1, U2.1 (OUT), U2.20 (OUT), U4.2 (VIN), U4.3 (EN)
- new net gpio: U5.1 (SDA), U5.12 (GPOUT), U5.2 (SCL)
- new net gpio?: U2.6 (~{PG}), U2.7 (STAT2), U2.8 (STAT1/~{LBO})

Commit message: fixing things
Parts:
- removed C35: C_Small, symbol Device:C_Small
- added C36: C_Small, symbol Device:C_Small
- added J6: Battery Connector, symbol Connector_Generic:Conn_01x02
- C30, C31: value 10 uF -> 10uF
- C32: value 0.1 uF -> 0.1uF
- C34: value 10 pF -> 10pF
- L1: value 1 uH -> 1uH
- R16: value 10KΩ -> 10K
- R17, R18: value 15KΩ -> 15K
- R19: value 1.2 M -> 1.2M
- R20: value 200 K -> 200k
- R21: value 10 K -> 10k
- R22: value 10 mΩ -> 10m
Connections:
- net USB_5V is gone; now on net VBUS: U2.17 (CE), U2.9 (~{TE})
- net GND: now also U5.3 (V_{SS}), C36.1, J6.2 (Pin_2); no longer R21.1, U5.5 (V_{DD})
- net VBAT renamed V_Batt
- net V_Batt: now also J6.1 (Pin_1)
- net V_3.3 renamed +3.3V
- net V_SYS renamed V_5V
- removed net gpio: U5.1 (SDA), U5.12 (GPOUT), U5.2 (SCL)
- removed net gpio?: U2.6 (~{PG}), U2.7 (STAT2), U2.8 (STAT1/~{LBO})
- new net: C36.2, R21.1, U5.5 (V_{DD})
- new net Monitor_GPOUT: U5.12 (GPOUT)
- new net Monitor_SCL: U5.2 (SCL)
- new net Monitor_SDA: U5.1 (SDA)
- new net Recharge_PG: U2.6 (~{PG})
- new net Recharge_ST1: U2.8 (STAT1/~{LBO})
- new net Recharge_ST2: U2.7 (STAT2)
- no-connect marks 0 -> 3
Other:
- moved on the sheet: R21

Commit message: Update LiPoPower_Module_Sheet.kicad_sch
Parts:
- added C35, C37, C38: 22uF, symbol Device:C_Small
Connections:
- net +3.3V: now also C35.2, C37.2, C38.2
- net GND: now also C35.1, C37.1, C38.1
Other:
- moved on the sheet: C30, C31, C32, C34, L1, R19, R20, U4

Commit message: push
Changed lines of the file:
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@@
 	(wire
 		(pts
-			(xy 217.17 49.53) (xy 223.52 49.53)
+			(xy 217.17 49.53) (xy 237.49 49.53)
 		)
 		(stroke
@@
 	(hierarchical_label "Monitor_GPOUT"
 		(shape input)
-		(at 223.52 49.53 0)
-		(effects
-			(font
+		(at 237.49 49.53 0)
+		(effects
+			(font

Commit message: Lotta changes
Parts:
- C30, C31, C32, C33, C34, C35, C36, C37, C38: footprint (none) -> Capacitor_SMD:C_0805_2012Metric_Pad1.18x1.45mm_HandSolder
- J6: footprint (none) -> PCB_Lib:JST Conn
- L1: footprint (none) -> Inductor_SMD:L_0805_2012Metric_Pad1.15x1.40mm_HandSolder
- R16, R17, R18, R19, R20, R21, R22: footprint (none) -> Resistor_SMD:R_0805_2012Metric_Pad1.20x1.40mm_HandSolder
Other:
- note added: "Inductor Size"
Changed lines of the file:
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@@
+		)
+	)
+	(text "Inductor Size"
+		(exclude_from_sim no)
+		(at 46.482 56.642 0)
+		(effects
+			(font
+				(size 1.27 1.27)
+			)
 		)
 	)
@@
 			)
 		)
-		(property "Footprint" ""
+		(property "Footprint" "Capacitor_SMD:C_0805_2012Metric_Pad1.18x1.45mm_HandSolder"
 			(at 219.71 39.37 0)
 			(effects
@@
 			)
 		)
-		(property "Footprint" ""
+		(property "Footprint" "Capacitor_SMD:C_0805_2012Metric_Pad1.18x1.45mm_HandSolder"
 			(at 100.33 35.56 0)
 			(effects
@@
 			)
 		)
-		(property "Footprint" ""
+		(property "Footprint" "Capacitor_SMD:C_0805_2012Metric_Pad1.18x1.45mm_HandSolder"
 			(at 109.22 97.79 0)
 			(effects
@@
 			)
 		)
-		(property "Footprint" ""
+		(property "Footprint" "Capacitor_SMD:C_0805_2012Metric_Pad1.18x1.45mm_HandSolder"
 			(at 91.44 35.56 0)
 			(effects
@@
 			)
 		)
-		(property "Footprint" ""
+		(property "Footprint" "Resistor_SMD:R_0805_2012Metric_Pad1.20x1.40mm_HandSolder"
 			(at 101.6 48.26 0)
 			(effects
@@
 			)
 		)
-		(property "Footprint" ""
+		(property "Footprint" "Resistor_SMD:R_0805_2012Metric_Pad1.20x1.40mm_HandSolder"
 			(at 33.02 118.11 0)
 			(effects
@@
 			)
 		)
-		(property "Footprint" ""
+		(property "Footprint" "Resistor_SMD:R_0805_2012Metric_Pad1.20x1.40mm_HandSolder"
 			(at 184.15 52.07 0)
 			(effects
@@
 			)
 		)
-		(property "Footprint" ""
+		(property "Footprint" "Resistor_SMD:R_0805_2012Metric_Pad1.20x1.40mm_HandSolder"
 			(at 24.13 118.11 0)
 			(effects
@@
 			)
 		)
-		(property "Footprint" ""
+		(property "Footprint" "Capacitor_SMD:C_0805_2012Metric_Pad1.18x1.45mm_HandSolder"
 			(at 111.76 48.26 0)
 			(effects
@@
 			)
 		)
-		(property "Footprint" ""
+		(property "Footprint" "Capacitor_SMD:C_0805_2012Metric_Pad1.18x1.45mm_HandSolder"
 			(at 43.18 40.64 0)
 			(effects
@@
 			)
 		)
-		(property "Footprint" ""
+		(property "Footprint" "Capacitor_SMD:C_0805_2012Metric_Pad1.18x1.45mm_HandSolder"
 			(at 34.29 40.64 0)
 			(effects
@@
 			)
 		)
-		(property "Footprint" ""
+		(property "Footprint" "Resistor_SMD:R_0805_2012Metric_Pad1.20x1.40mm_HandSolder"
 			(at 41.91 118.11 0)
 			(effects
@@
 			)
 		)
-		(property "Footprint" ""
+		(property "Footprint" "Resistor_SMD:R_0805_2012Metric_Pad1.20x1.40mm_HandSolder"
 			(at 83.82 40.64 0)
 			(effects
@@
 			)
 		)
-		(property "Footprint" ""
+		(property "Footprint" "Capacitor_SMD:C_0805_2012Metric_Pad1.18x1.45mm_HandSolder"
 			(at 107.95 35.56 0)
 			(effects
@@
 			)
 		)
-		(property "Footprint" ""
+		(property "Footprint" "Inductor_SMD:L_0805_2012Metric_Pad1.15x1.40mm_HandSolder"
 			(at 57.15 53.34 0)
 			(effects
@@
 			)
 		)
-		(property "Footprint" ""
+		(property "Footprint" "PCB_Lib:JST Conn"
 			(at 125.73 111.76 0)
 			(effects
@@
 			)
 		)
-		(property "Footprint" ""
+		(property "Footprint" "Resistor_SMD:R_0805_2012Metric_Pad1.20x1.40mm_HandSolder"
 			(at 181.61 68.58 0)
 			(effects
@@
 			)
 		)
-		(property "Footprint" ""
+		(property "Footprint" "Capacitor_SMD:C_0805_2012Metric_Pad1.18x1.45mm_HandSolder"
 			(at 87.63 55.88 0)
 			(effects

Commit message: onto PCB
Changed lines of the file:
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@@
-		)
-	)
-	(global_label "VBUS"
-		(shape input)
-		(at 26.67 95.25 180)
-		(fields_autoplaced yes)
-		(effects
-			(font
-				(size 1.27 1.27)
-			)
-			(justify right)
-		)
-		(property "Intersheetrefs" "${INTERSHEET_REFS}"
-			(at 18.7862 95.25 0)
-			(effects
-				(font
-					(size 1.27 1.27)
-				)
-				(justify right)
-				(hide yes)
-			)
 		)
 	)
@@
 					(unit 1)
 				)
+			)
+		)
+	)
+	(symbol
+		(lib_id "power:VBUS")
+		(at 26.67 95.25 0)
+		(unit 1)
+		(exclude_from_sim no)
+		(in_bom yes)
+		(on_board yes)
+		(dnp no)
+		(fields_autoplaced yes)
+		(property "Reference" "#PWR037"
+			(at 26.67 99.06 0)
+			(effects
+				(font
+					(size 1.27 1.27)
+				)
+				(hide yes)
+			)
+		)
+		(property "Value" "VBUS"
+			(at 26.67 90.17 0)
+			(effects
+				(font
+					(size 1.27 1.27)
+				)
+			)
+		)
+		(property "Footprint" ""
+			(at 26.67 95.25 0)
+			(effects
+				(font
+					(size 1.27 1.27)
+				)
+				(hide yes)
+			)
+		)
+		(property "Datasheet" ""
+			(at 26.67 95.25 0)
+			(effects
+				(font
+					(size 1.27 1.27)
+				)
+				(hide yes)
+			)
+		)
+		(property "Description" "Power symbol creates a global label with name \"VBUS\""
+			(at 26.67 95.25 0)
+			(effects
+				(font
+					(size 1.27 1.27)
+				)
+				(hide yes)
+			)
+		)
+		(pin "1"
+		)
+		(instances
+			(project ""
+				(path "/527ae649-08be-4368-9cf9-441ebba18eca/b7e4818e-74b8-4bbc-96b7-b26a83655ade"
+					(reference "#PWR037")
+					(unit 1)
+				)

Commit message: power & power pcb layout
Parts:
- C33: value C_Small -> 4.7 uF
- C36: value C_Small -> 0.47uF
- L1: footprint Inductor_SMD:L_0805_2012Metric_Pad1.15x1.40mm_HandSolder -> Inductor_SMD:L_1008_2520Metric_Pad1.43x2.20mm_HandSolder
Other:
- note added: "rscl & rsda"
Changed lines of the file:
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@@
+		)
+	)
+	(text "rscl & rsda\n"
+		(exclude_from_sim no)
+		(at 179.07 29.21 0)
+		(effects
+			(font
+				(size 1.27 1.27)
+			)
+		)
+	)
+	(label "cbat add"
+		(at 173.99 34.29 0)
+		(effects
+			(font
+				(size 1.27 1.27)
+			)
+			(justify left bottom)
 		)
 	)
@@
 			)
 		)
-		(property "Value" "C_Small"
+		(property "Value" "0.47uF"
 			(at 222.25 40.6462 0)
 			(effects
@@
 			)
 		)
-		(property "Value" "C_Small"
+		(property "Value" "4.7 uF"
 			(at 111.76 99.0662 0)
 			(effects
@@
 			)
 		)
-		(property "Footprint" "Inductor_SMD:L_0805_2012Metric_Pad1.15x1.40mm_HandSolder"
+		(property "Footprint" "Inductor_SMD:L_1008_2520Metric_Pad1.43x2.20mm_HandSolder"
 			(at 57.15 53.34 0)
 			(effects

Commit message: layout and coulomb counter sch update
Connections:
- net GND: now also C36.2, R21.1; no longer C36.1
- new net: C36.1, U5.5 (V_{DD})
Other:
- moved on the sheet: C36
Changed lines of the file:
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@@
 	)
 	(junction
-		(at 219.71 41.91)
-		(diameter 0)
-		(color 0 0 0 0)
-	)
-	(junction
 		(at 119.38 111.76)
 		(diameter 0)
@@
 	)
 	(junction
+		(at 201.93 67.31)
+		(diameter 0)
+		(color 0 0 0 0)
+	)
+	(junction
 		(at 24.13 123.19)
 		(diameter 0)
@@
 	)
 	(junction
+		(at 231.14 67.31)
+		(diameter 0)
+		(color 0 0 0 0)
+	)
+	(junction
 		(at 91.44 38.1)
 		(diameter 0)
@@
 	(wire
 		(pts
-			(xy 231.14 41.91) (xy 231.14 77.47)
+			(xy 69.85 66.04) (xy 68.58 66.04)
 		)
 		(stroke
@@
 	(wire
 		(pts
-			(xy 69.85 66.04) (xy 68.58 66.04)
+			(xy 231.14 41.91) (xy 231.14 67.31)
 		)
 		(stroke
@@
 	(wire
 		(pts
+			(xy 201.93 69.85) (xy 201.93 67.31)
+		)
+		(stroke
+			(width 0)
+			(type default)
+		)
+	)
+	(wire
+		(pts
 			(xy 43.18 45.72) (xy 34.29 45.72)
 		)
@@
 	(wire
 		(pts
+			(xy 217.17 41.91) (xy 222.25 41.91)
+		)
+		(stroke
+			(width 0)
+			(type default)
+		)
+	)
+	(wire
+		(pts
 			(xy 24.13 105.41) (xy 24.13 115.57)
 		)
@@
 	(wire
 		(pts
+			(xy 227.33 41.91) (xy 231.14 41.91)
+		)
+		(stroke
+			(width 0)
+			(type default)
+		)
+	)
+	(wire
+		(pts
 			(xy 49.53 100.33) (xy 21.59 100.33)
 		)
@@
 	(wire
 		(pts
-			(xy 85.09 102.87) (xy 88.9 102.87)
+			(xy 201.93 67.31) (xy 231.14 67.31)
 		)
 		(stroke
@@
 	(wire
 		(pts
-			(xy 83.82 38.1) (xy 91.44 38.1)
+			(xy 85.09 102.87) (xy 88.9 102.87)
 		)
 		(stroke
@@
 	(wire
 		(pts
-			(xy 219.71 41.91) (xy 231.14 41.91)
+			(xy 83.82 38.1) (xy 91.44 38.1)
 		)
 		(stroke
@@
 	(wire
 		(pts
+			(xy 231.14 67.31) (xy 231.14 77.47)
+		)
+		(stroke
+			(width 0)
+			(type default)
+		)
+	)
+	(wire
+		(pts
 			(xy 181.61 77.47) (xy 231.14 77.47)
 		)
@@
 	(wire
 		(pts
-			(xy 107.95 38.1) (xy 118.11 38.1)
+			(xy 201.93 67.31) (xy 201.93 64.77)
 		)
 		(stroke
@@
 	(wire
 		(pts
-			(xy 181.61 59.69) (xy 186.69 59.69)
+			(xy 107.95 38.1) (xy 118.11 38.1)
 		)
 		(stroke
@@
 	(wire
 		(pts
-			(xy 163.83 39.37) (xy 186.69 39.37)
+			(xy 181.61 59.69) (xy 186.69 59.69)
 		)
 		(stroke
@@
 	(wire
 		(pts
-			(xy 41.91 120.65) (xy 41.91 123.19)
+			(xy 163.83 39.37) (xy 186.69 39.37)
 		)
 		(stroke
@@
 	(wire
 		(pts
-			(xy 69.85 66.04) (xy 71.12 66.04)
+			(xy 41.91 120.65) (xy 41.91 123.19)
 		)
 		(stroke
@@
 	(wire
 		(pts
-			(xy 60.96 43.18) (xy 55.88 43.18)
+			(xy 69.85 66.04) (xy 71.12 66.04)
 		)
 		(stroke
@@
 	(wire
 		(pts
-			(xy 106.68 111.76) (xy 119.38 111.76)
+			(xy 60.96 43.18) (xy 55.88 43.18)
 		)
 		(stroke
@@
 	(wire
 		(pts
-			(xy 217.17 41.91) (xy 219.71 41.91)
+			(xy 106.68 111.76) (xy 119.38 111.76)
 		)
 		(stroke
@@
 	(symbol
 		(lib_id "Device:C_Small")
-		(at 219.71 39.37 0)
+		(at 224.79 41.91 90)
 		(unit 1)
 		(exclude_from_sim no)
@@
 		(fields_autoplaced yes)
 		(property "Reference" "C36"
-			(at 222.25 38.1062 0)
+			(at 223.5262 39.37 0)
 			(effects
 				(font
@@
 		)
 		(property "Value" "0.47uF"
-			(at 222.25 40.6462 0)
+			(at 226.0662 39.37 0)
 			(effects
 				(font
@@
 		)
 		(property "Footprint" "Capacitor_SMD:C_0805_2012Metric_Pad1.18x1.45mm_HandSolder"
-			(at 219.71 39.37 0)
+			(at 224.79 41.91 0)
 			(effects
 				(font
@@
 		)
 		(property "Datasheet" "~"
-			(at 219.71 39.37 0)
+			(at 224.79 41.91 0)
 			(effects
 				(font
@@
 		)
 		(property "Description" "Unpolarized capacitor, small symbol"
-			(at 219.71 39.37 0)
+			(at 224.79 41.91 0)
 			(effects
 				(font
@@
 	(symbol
 		(lib_id "power:GND")
-		(at 219.71 36.83 180)
-		(unit 1)
-		(exclude_from_sim no)
-		(in_bom yes)
-		(on_board yes)
-		(dnp no)
-		(fields_autoplaced yes)
-		(property "Reference" "#PWR032"
-			(at 219.71 30.48 0)
-			(effects
-				(font
-					(size 1.27 1.27)
-				)
-				(hide yes)
-			)
-		)
-		(property "Value" "GND"
-			(at 219.71 31.75 0)
-			(effects
-				(font
-					(size 1.27 1.27)
-				)
-			)
-		)
-		(property "Footprint" ""
-			(at 219.71 36.83 0)
-			(effects
-				(font
-					(size 1.27 1.27)
-				)
-				(hide yes)
-			)
-		)
-		(property "Datasheet" ""
-			(at 219.71 36.83 0)
-			(effects
-				(font
-					(size 1.27 1.27)
-				)
-				(hide yes)
-			)
-		)
-		(property "Description" "Power symbol creates a global label with name \"GND\" , ground"
-			(at 219.71 36.83 0)
-			(effects
-				(font
-					(size 1.27 1.27)
-				)
-				(hide yes)
-			)
-		)
-		(pin "1"
-		)
-		(instances
-			(project ""
-				(path "/527ae649-08be-4368-9cf9-441ebba18eca/b7e4818e-74b8-4bbc-96b7-b26a83655ade"
-					(reference "#PWR032")
-					(unit 1)
-				)
-			)
-		)
-	)
-	(symbol
-		(lib_id "power:GND")
 		(at 67.31 133.35 0)
 		(unit 1)
@@
 	(symbol
 		(lib_id "power:GND")
-		(at 201.93 64.77 0)
+		(at 201.93 69.85 0)
 		(unit 1)
 		(exclude_from_sim no)
@@
 		(fields_autoplaced yes)
 		(property "Reference" "#PWR033"
-			(at 201.93 71.12 0)
+			(at 201.93 76.2 0)
 			(effects
 				(font
@@
 		)
 		(property "Value" "GND"
-			(at 201.93 69.85 0)
+			(at 201.93 74.93 0)
 			(effects
 				(font
@@
 		)
 		(property "Footprint" ""
-			(at 201.93 64.77 0)
+			(at 201.93 69.85 0)
 			(effects
 				(font
@@
 		)
 		(property "Datasheet" ""
-			(at 201.93 64.77 0)
+			(at 201.93 69.85 0)
 			(effects
 				(font
@@
 		)
 		(property "Description" "Power symbol creates a global label with name \"GND\" , ground"
-			(at 201.93 64.77 0)
+			(at 201.93 69.85 0)
 			(effects
 				(font
