File: EInkDisplay-PCB/ECE477-SeniorDesign/LiPoPower_Module_Sheet.kicad_sch (KiCad schematic)
At the start: 21 parts, among them J6 Battery Connector, U2 MCP73871, U4 TPS63060, U5 BQ27441-G1

Commit message: Update LiPoPower_Module_Sheet.kicad_sch
Parts:
- removed R21: 10k, Resistor_SMD:R_0805_2012Metric_Pad1.20x1.40mm_HandSolder, symbol Device:R_Small_US
- added R2, R3, R4: 10k, Resistor_SMD:R_0805_2012Metric_Pad1.20x1.40mm_HandSolder, symbol Device:R_Small_US
Connections:
- net GND: now also U5.10 (BIN)
- net Monitor_GPOUT: now also R4.2
- net Monitor_SCL: no longer names the net of U5.2 (SCL)
- net Monitor_SCL: now also R3.2
- net Monitor_SDA: no longer names the net of U5.1 (SDA)
- net Monitor_SDA: now also R2.2
- new net 3.3V: R2.1, R3.1, R4.1
Other:
- note removed: "rscl & rsda"

Commit message: changes
Changed lines of the file:
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@@
-		)
-	)
-	(label "cbat add"
-		(at 176.53 27.94 0)
-		(effects
-			(font
-				(size 1.27 1.27)
-			)
-			(justify left bottom)
 		)
 	)

Commit message: pushing
Connections:
- net +3.3V: now also R2.2, R3.2, R4.1
- net Monitor_SDA: now reaches U5.1 (SDA)
- net Monitor_SDA: now also R2.1; no longer R2.2
- net Monitor_SCL: now reaches U5.2 (SCL)
- net Monitor_SCL: now also R3.1; no longer R3.2
- removed net 3.3V: R2.1, R3.1, R4.1
Other:
- moved on the sheet: R2, R3

Commit message: pushing
Parts:
- renumbered C30 to C19, C31 to C20, C32 to C21, C35 to C22, C37 to C23, C38 to C24, C33 to C25, C34 to C26, C36 to C27, J6 to J3, R4 to R10, R16 to R2, R17 to R3, R18 to R4, R19 to R5, R20 to R6, R3 to R7, R2 to R8, R22 to R9, U2 to U3
