File: EInkDisplay-PCB/ECE477-SeniorDesign/LiPoPower_Module_Sheet.kicad_sch (KiCad schematic)
At the start: 32 parts, among them J6 Battery Connector, U4 TPS63060, U5 BQ27441-G1, U6 MCP73871-2CCI/ML

Commit message: push
Parts:
- removed D1, D2, D3: LED_Small, LED_SMD:LED_0805_2012Metric, symbol Device:LED_Small
- removed R10, R12, R13: 470, Resistor_SMD:R_0805_2012Metric_Pad1.20x1.40mm_HandSolder, symbol Device:R_Small_US
Connections:
- net VBUS: now also U6.2 (VPCC), U6.9 (*TE)
- net V_Batt: no longer U6.2 (VPCC), U6.9 (*TE)

Commit message: again
Parts:
- added C25: 1uF, Capacitor_SMD:C_0805_2012Metric_Pad1.18x1.45mm_HandSolder, symbol Device:C_Small
- added R3: 1.8M, Resistor_SMD:R_0805_2012Metric_Pad1.20x1.40mm_HandSolder, symbol Device:R_Small_US
Connections:
- net +3.3V: now also R3.1
- net GND: now also C25.2; no longer U5.10 (BIN)
- net V_Batt: now also R11.2, U5.7 (SRN); no longer R11.1, U5.6 (BAT), U5.8 (SRP)
- new net: R3.2, U5.10 (BIN)
- new net BATTERY_IN: C25.1, R11.1, U5.6 (BAT), U5.8 (SRP)
Other:
- moved on the sheet: R11

Commit message: pusj
Connections:
- net BATTERY_IN: now also J6.1 (Pin_1)
- net V_Batt: no longer J6.1 (Pin_1)
Other:
- moved on the sheet: C28, C29, C30, J6, R14, R16, R17, R18, U6

Commit message: done
Parts:
- U4: footprint Package_SON:Texas_S-PWSON-N10_ThermalVias -> PCB_Lib:DSC0010E
Changed lines of the file:
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@@
 			)
 		)
-		(property "Footprint" "Package_SON:Texas_S-PWSON-N10_ThermalVias"
+		(property "Footprint" "PCB_Lib:DSC0010E"
 			(at 71.12 64.77 0)
 			(effects

Commit message: Regulator footprint and sch update
Parts:
- removed C21: 0.1uF, Capacitor_SMD:C_0805_2012Metric_Pad1.18x1.45mm_HandSolder, symbol Device:C_Small
- removed C22, C23, C24: 22uF, Capacitor_SMD:C_0805_2012Metric_Pad1.18x1.45mm_HandSolder, symbol Device:C_Small
- removed C26: 10pF, Capacitor_SMD:C_0805_2012Metric_Pad1.18x1.45mm_HandSolder, symbol Device:C_Small
- removed U4: TPS63060, PCB_Lib:DSC0010E, symbol Regulator_Switching:TPS63060
- added R4: 91k, Resistor_SMD:R_0805_2012Metric_Pad1.20x1.40mm_HandSolder, symbol Device:R_Small_US
- added U10: TPS63802DLA, Project_PCB_Library:TPS63802DLR, symbol Regulator_Switching:TPS63060
- C20: value 10uF -> 22uF
- L1: value 1uH -> 470nH; footprint Inductor_SMD:L_1008_2520Metric_Pad1.43x2.20mm_HandSolder -> Project_PCB_Library:IND_XFL4015_COC-L
- R6: value 1.2M -> 100k
- R7: value 200k -> 511k
Connections:
- net +3.3V: now also C20.1, R7.1, U10.6 (VOUT)
- net GND: now also R4.2, U10.2 (MODE), U10.3 (AGND), U10.8 (GND); no longer R7.2
- net V_5V: now also U10.1 (EN), U10.10 (VIN); no longer C20.1
- net at L1.1: now also U10.9 (L1)
- net at L1.2: now also U10.7 (L2)
- net at R6.2: now also U10.4 (PG); no longer R7.1
- new net: R4.1, R7.2, U10.5 (FB)
- no-connect marks 2 -> 1
Other:
- note removed: "Inductor Size"
- moved on the sheet: C19, C20, L1, R6, R7

Commit message: push
Connections:
- net +3.3V: no longer R6.1
- net V_5V: now also R6.2
- net at U10.4 (PG): now also R6.1; no longer R6.2
Other:
- moved on the sheet: R6
Changed lines of the file:
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@@
 	(paper "A1")
 	(junction
-		(at 77.47 40.64)
-		(diameter 0)
-		(color 0 0 0 0)
-	)
-	(junction
 		(at 162.56 39.37)
 		(diameter 0)
@@
 	(wire
 		(pts
-			(xy 72.39 45.72) (xy 77.47 45.72)
+			(xy 72.39 45.72) (xy 78.74 45.72)
 		)
 		(stroke
@@
 	(wire
 		(pts
+			(xy 72.39 39.37) (xy 72.39 40.64)
+		)
+		(stroke
+			(width 0)
+			(type default)
+		)
+	)
+	(wire
+		(pts
 			(xy 179.07 50.8) (xy 186.69 50.8)
 		)
@@
 	(wire
 		(pts
+			(xy 78.74 34.29) (xy 78.74 40.64)
+		)
+		(stroke
+			(width 0)
+			(type default)
+		)
+	)
+	(wire
+		(pts
 			(xy 153.67 130.81) (xy 156.21 130.81)
 		)
@@
 	(wire
 		(pts
+			(xy 87.63 39.37) (xy 87.63 40.64)
+		)
+		(stroke
+			(width 0)
+			(type default)
+		)
+	)
+	(wire
+		(pts
 			(xy 217.17 41.91) (xy 222.25 41.91)
 		)
@@
 	(wire
 		(pts
-			(xy 77.47 40.64) (xy 87.63 40.64)
-		)
-		(stroke
-			(width 0)
-			(type default)
-		)
-	)
-	(wire
-		(pts
 			(xy 67.31 120.65) (xy 63.5 120.65)
 		)
@@
 	(wire
 		(pts
-			(xy 72.39 40.64) (xy 77.47 40.64)
+			(xy 72.39 39.37) (xy 87.63 39.37)
 		)
 		(stroke
@@
 		)
 	)
+	(global_label "V_5V"
+		(shape input)
+		(at 78.74 34.29 0)
+		(fields_autoplaced yes)
+		(effects
+			(font
+				(size 1.27 1.27)
+			)
+			(justify left)
+		)
+		(property "Intersheetrefs" "${INTERSHEET_REFS}"
+			(at 86.0795 34.29 0)
+			(effects
+				(font
+					(size 1.27 1.27)
+				)
+				(justify left)
+				(hide yes)
+			)
+		)
+	)
 	(global_label "V_Batt"
 		(shape input)
@@
 	(symbol
 		(lib_id "Device:R_Small_US")
-		(at 77.47 43.18 0)
+		(at 78.74 43.18 180)
 		(unit 1)
 		(exclude_from_sim no)
@@
 		(fields_autoplaced yes)
 		(property "Reference" "R6"
-			(at 80.01 41.9099 0)
+			(at 81.28 41.9099 0)
 			(effects
 				(font
 					(size 1.27 1.27)
 				)
-				(justify left)
+				(justify right)
 			)
 		)
 		(property "Value" "100k"
-			(at 80.01 44.4499 0)
+			(at 81.28 44.4499 0)
 			(effects
 				(font
 					(size 1.27 1.27)
 				)
-				(justify left)
+				(justify right)
 			)
 		)
 		(property "Footprint" "Resistor_SMD:R_0805_2012Metric_Pad1.20x1.40mm_HandSolder"
-			(at 77.47 43.18 0)
+			(at 78.74 43.18 0)
 			(effects
 				(font
@@
 		)
 		(property "Datasheet" "~"
-			(at 77.47 43.18 0)
+			(at 78.74 43.18 0)
 			(effects
 				(font
@@
 		)
 		(property "Description" "Resistor, small US symbol"
-			(at 77.47 43.18 0)
+			(at 78.74 43.18 0)
 			(effects
 				(font

Commit message: push
Connections:
- net GND: now also U5.13 (PAD)
- no-connect marks 1 -> 0
Changed lines of the file:
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@@
 		(color 0 0 0 0)
 	)
-	(no_connect
-		(at 199.39 64.77)
-	)
 	(wire
 		(pts
@@
 	(wire
 		(pts
+			(xy 199.39 67.31) (xy 201.93 67.31)
+		)
+		(stroke
+			(width 0)
+			(type default)
+		)
+	)
+	(wire
+		(pts
 			(xy 38.1 40.64) (xy 40.64 40.64)
 		)
@@
 		)
 		(stroke
+			(width 0)
+			(type default)
+		)
+	)
+	(wire
+		(pts
+			(xy 199.39 64.77) (xy 199.39 67.31)
+		)
+		(stroke

Commit message: push
Parts:
- J6: footprint PCB_Lib:JST Conn -> Connector_JST:JST_PH_S2B-PH-SM4-TB_1x02-1MP_P2.00mm_Horizontal
Changed lines of the file:
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@@
 			)
 		)
-		(property "Footprint" "PCB_Lib:JST Conn"
+		(property "Footprint" "Connector_JST:JST_PH_S2B-PH-SM4-TB_1x02-1MP_P2.00mm_Horizontal"
 			(at 248.92 64.77 0)
 			(effects
