File: EInkDisplay-PCB/ECE477-SeniorDesign/ECE477-SeniorDesign.kicad_pcb (KiCad board)
At the start: 2 copper layers, 103.8 x 82.5 mm, 95 parts, among them J3 JST Conn, J4 JST Conn, J5 JST Conn, J6 Battery Connector, J9 Micro_SD_Card_Det1, U1 CP2102-GMR, U2 MCP73871, U3 STM32L496ZGTxP, U4 TPS63060, U5 BQ27441-G1, U6 NUP2202, U7 PTS526 SK15 SMTR2 LFS, U9 74LVC125APW_118, Y1 Y1

Commit message: pushing
Parts:
- removed C21: 100nF, Capacitor_SMD:C_0805_2012Metric_Pad1.18x1.45mm_HandSolder
- added J2: Conn_01x05_Pin, Connector_PinHeader_1.00mm:PinHeader_1x05_P1.00mm_Vertical, F.Cu at (143.5, 47.0)
- moved C20 68.5 mm to (140.2, 101.8), turned to 0 degrees
- moved C10 27.6 mm to (166.0, 93.4), turned to -90 degrees
- moved U7 4.83 mm to (139.5, 107.8), turned to -90 degrees
Connections:
- R2 pad 1: 3.3V -> /LipoPower/Monitor_SDA
- R2 pad 2: Net-(U5-SDA) -> +3.3V
- R3 pad 1: 3.3V -> /LipoPower/Monitor_SCL
- R3 pad 2: Net-(U5-SCL) -> +3.3V
- R4 pad 1: 3.3V -> +3.3V
- U1 pad 4: Net-(Je1-D+) -> Net-(J1-D+)
- U1 pad 5: Net-(Je1-D-) -> Net-(J1-D-)
- U3 pad 1: /ExtraPeriphs/button3 -> /ExtraPeriphs/button1
- U3 pad 135: unconnected-(U3-PB6-Pad135) -> Extra_5
- U3 pad 136: unconnected-(U3-PB7-Pad136) -> Extra_4
- U3 pad 138: unconnected-(U3-PB8-Pad138) -> Extra_3
- U3 pad 140: Extra_1 -> Extra_2
- U3 pad 141: Extra_2 -> Extra_1
- U3 pad 3: /ExtraPeriphs/button1 -> /ExtraPeriphs/button3
- U3 pad 81: 3.3V -> /LipoPower/Monitor_SCL
- U3 pad 82: 3.3V -> /LipoPower/Monitor_SDA
- U5 pad 1: Net-(U5-SDA) -> /LipoPower/Monitor_SDA
- U5 pad 2: Net-(U5-SCL) -> /LipoPower/Monitor_SCL
- U6 pad 1: Net-(Je1-D+) -> Net-(J1-D+)
- U6 pad 6: Net-(Je1-D-) -> Net-(J1-D-)
Routing:
- net Extra_2: track 0.00 -> 48.9 mm
- net Extra_1: track 0.00 -> 42.5 mm
- net Extra_3: track 0.00 -> 36.1 mm, vias 0 -> 1
- net Extra_4: track 0.00 -> 35.6 mm, vias 0 -> 1
- net Extra_5: track 0.00 -> 35.5 mm, vias 0 -> 1
- net /ExtraPeriphs/button1: track 0.00 -> 24.0 mm
- net GND: track 29.9 -> 48.9 mm, vias 2 -> 14
- net /ExtraPeriphs/button2: track 2.13 -> 19.6 mm
- net NRST: track 0.00 -> 15.5 mm
- net /ExtraPeriphs/button3: track 2.24 -> 16.0 mm

Commit message: Layout update
Parts:
- removed the ? at (165.8, 118.2)
- removed Je1: USB_B, Connector_USB:USB_B_TE_5787834_Vertical
- added ?: , , F.Cu at (163.5, 108.1)
- added ?: , , F.Cu at (164.8, 111.2)
- added ?: , , F.Cu at (158.1, 107.4)
- added ?: , , F.Cu at (162.7, 109.4)
- added J1: USB_A, Connector_USB:USB_A_Receptacle_GCT_USB1046, F.Cu at (196.5, 87.7)
- moved R20 20.5 mm to (155.3, 109.0), turned to 180 degrees
- moved C38 20.3 mm to (154.2, 114.1), turned to 90 degrees
- moved R19 19.0 mm to (155.3, 110.9), turned to 0 degrees
- moved C8 16.9 mm to (174.2, 93.2)
- moved C6 16.6 mm to (174.2, 95.3)
- moved C37 16.3 mm to (156.2, 114.1), turned to 90 degrees
- moved U6 15.3 mm to (183.1, 83.0)
- moved C34 14.2 mm to (158.2, 110.3), turned to 90 degrees
- moved C32 12.9 mm to (161.2, 108.2), turned to 0 degrees
- moved C35 12.3 mm to (158.2, 114.1), turned to 90 degrees
- moved R4 11.6 mm to (181.2, 110.6), turned to 0 degrees
- moved ? 10.00 mm to (162.0, 109.4), turned to 180 degrees
- moved ? 9.56 mm to (161.6, 109.9), turned to 180 degrees
- moved R2 9.11 mm to (175.7, 110.1), turned to 90 degrees
- moved R3 9.11 mm to (173.7, 110.1), turned to 90 degrees
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Connections:
- net Net-(J1-D+) renamed /USB-UART/D_P
- net Net-(J1-D-) renamed /USB-UART/D_N
Routing:
- net GND: track 48.9 -> 63.5 mm, vias 14 -> 15
- net /USB-UART/D_P: track 0.00 -> 10.8 mm
- net /USB-UART/D_N: track 0.00 -> 10.4 mm
- net +3.3V: track 31.6 -> 38.0 mm
- net Net-(U4-FB): track 0.00 -> 6.28 mm
- net Net-(U4-L1): track 0.00 -> 5.73 mm
- net Net-(U4-L2): track 0.00 -> 5.61 mm
- net V_5V: track 0.00 -> 5.37 mm
- net /LipoPower/Monitor_SCL: track 0.00 -> 5.07 mm
- net Net-(U4-VAUX): track 0.00 -> 3.85 mm
- net /LipoPower/Monitor_SDA: track 0.00 -> 2.78 mm
- added copper zone on F.Cu, net GND

Commit message: pushing
Parts:
- added C21: 10pF, Capacitor_SMD:C_0805_2012Metric_Pad1.18x1.45mm_HandSolder, F.Cu at (130.8, 103.0)
- added C39: 100n, Capacitor_SMD:C_0805_2012Metric_Pad1.18x1.45mm_HandSolder, F.Cu at (133.0, 103.0)
- added D5: 1N4148, Diode_THT:D_DO-35_SOD27_P7.62mm_Horizontal, F.Cu at (124.8, 55.9)
- added J8: JST Conn, PCB_Lib:JST Conn, F.Cu at (116.5, 99.2)
- added R5: 100k, Resistor_SMD:R_0805_2012Metric_Pad1.20x1.40mm_HandSolder, F.Cu at (124.3, 101.0)
- added R6: 1k, Resistor_SMD:R_0805_2012Metric_Pad1.20x1.40mm_HandSolder, F.Cu at (131.8, 100.0)
- D1, D2, D3: value D -> 1N4148; footprint Diode_SMD:D_0805_2012Metric_Pad1.15x1.40mm_HandSolder -> Diode_THT:D_DO-35_SOD27_P7.62mm_Horizontal
- moved D3 12.8 mm to (132.0, 97.5)
- moved D2 10.4 mm to (131.8, 83.5)
- moved D1 10.3 mm to (131.6, 72.2)
Connections:
- C22 pad 1: Net-(D1-K) -> Net-(D5-K)
- C24 pad 1: Net-(D2-K) -> Net-(D1-K)
- C26 pad 1: Net-(D3-K) -> Net-(D2-K)
- J3 pad 2: Net-(D1-A) -> Net-(D5-A)
- J4 pad 2: Net-(D2-A) -> Net-(D1-A)
- J5 pad 2: Net-(D3-A) -> Net-(D2-A)
- R10 pad 1: Net-(D1-A) -> Net-(D5-A)
- R11 pad 1: Net-(D1-K) -> Net-(D5-K)
- R12 pad 1: Net-(D2-A) -> Net-(D1-A)
- R13 pad 1: Net-(D2-K) -> Net-(D1-K)
- R14 pad 1: Net-(D3-A) -> Net-(D2-A)
- R15 pad 1: Net-(D3-K) -> Net-(D2-K)
- U3 pad 4: unconnected-(U3-PE5-Pad4) -> /ExtraPeriphs/switch
Routing:
- net /ExtraPeriphs/switch: track 0.00 -> 27.4 mm, vias 0 -> 2
- net Net-(D5-K): track 0.00 -> 12.7 mm
- net Net-(D1-A): track 0.00 -> 9.08 mm
- net Net-(D1-K): track 0.00 -> 7.59 mm
- net GND: track 63.5 -> 71.0 mm, vias 15 -> 20
- net Net-(D5-A): track 0.00 -> 5.78 mm
- net Net-(D2-A): track 5.94 -> 9.37 mm
- net Net-(D2-K): track 3.85 -> 6.94 mm
- net /ExtraPeriphs/button1: track 24.0 -> 26.4 mm
- net Net-(D3-K): track 3.67 -> 4.94 mm

Commit message: pushing
Parts:
- removed the R21 at (187.5, 125.2)
- added J10: Conn_01x05_Pin, Connector_PinHeader_1.00mm:PinHeader_1x05_P1.00mm_Vertical, F.Cu at (180.2, 47.0)
- added J11: Conn_01x05_Pin, Connector_PinHeader_1.00mm:PinHeader_1x05_P1.00mm_Vertical, F.Cu at (173.5, 47.0)
- added TP1: UART_TX, TestPoint:TestPoint_Pad_1.0x1.0mm, F.Cu at (169.0, 84.5)
- added TP10: ~, TestPoint:TestPoint_Pad_1.0x1.0mm, F.Cu at (59.9, 59.3)
- added TP11: ~, TestPoint:TestPoint_Pad_1.0x1.0mm, F.Cu at (59.9, 63.4)
- added TP12: ~, TestPoint:TestPoint_Pad_1.0x1.0mm, F.Cu at (59.9, 67.4)
- added TP13: NSRT, TestPoint:TestPoint_Pad_1.0x1.0mm, F.Cu at (59.9, 71.5)
- added TP14: BOOT0, TestPoint:TestPoint_Pad_1.0x1.0mm, F.Cu at (59.9, 75.5)
- added TP15: ~, TestPoint:TestPoint_Pad_1.0x1.0mm, F.Cu at (132.2, 49.5)
- added TP16: ~, TestPoint:TestPoint_Pad_1.0x1.0mm, F.Cu at (64.0, 59.3)
- added TP17: ~, TestPoint:TestPoint_Pad_1.0x1.0mm, F.Cu at (64.0, 63.4)
- added TP18: ~, TestPoint:TestPoint_Pad_1.0x1.0mm, F.Cu at (64.0, 67.4)
- added TP19: ~, TestPoint:TestPoint_Pad_1.0x1.0mm, F.Cu at (64.0, 71.5)
- added TP2: UART_RX, TestPoint:TestPoint_Pad_1.0x1.0mm, F.Cu at (173.2, 90.8)
- added TP20: ~, TestPoint:TestPoint_Pad_1.0x1.0mm, F.Cu at (64.0, 75.5)
- added TP21: ~, TestPoint:TestPoint_Pad_1.0x1.0mm, F.Cu at (144.8, 51.5)
- added TP22: ~, TestPoint:TestPoint_Pad_1.0x1.0mm, F.Cu at (144.8, 49.2)
- added TP23: ~, TestPoint:TestPoint_Pad_1.0x1.0mm, F.Cu at (144.8, 53.8)
- added TP24: ~, TestPoint:TestPoint_Pad_1.0x1.0mm, F.Cu at (191.8, 63.2)
- added TP25: ~, TestPoint:TestPoint_Pad_1.0x1.0mm, F.Cu at (68.0, 71.5)
- added TP27: VBUS, TestPoint:TestPoint_Pad_1.0x1.0mm, F.Cu at (181.0, 77.0)
- added TP3: E_MOSI, TestPoint:TestPoint_Pad_1.0x1.0mm, F.Cu at (146.5, 106.2)
- added TP4: E_NSS, TestPoint:TestPoint_Pad_1.0x1.0mm, F.Cu at (147.0, 111.0)
- added TP5: E_RST, TestPoint:TestPoint_Pad_1.0x1.0mm, F.Cu at (127.5, 112.0)
- added TP6: E_SCK, TestPoint:TestPoint_Pad_1.0x1.0mm, F.Cu at (127.5, 116.0)
- added TP7: E_D/C, TestPoint:TestPoint_Pad_1.0x1.0mm, F.Cu at (131.5, 112.0)
- added TP8: E_Busy, TestPoint:TestPoint_Pad_1.0x1.0mm, F.Cu at (131.5, 116.0)
- added TP9: ~, TestPoint:TestPoint_Pad_1.0x1.0mm, F.Cu at (154.0, 73.0)
- SWBOOT1: renamed from SWBOOT0; footprint PCB_Lib:PCM12SMTR_CNK -> Button_Switch_SMD:SW_SPDT_PCM12
- moved C31 15.0 mm to (175.7, 78.2)
- moved C29 14.9 mm to (175.7, 80.5)
- moved C28 14.4 mm to (180.3, 81.0)
- moved H4 13.4 mm to (200.0, 120.0)
- moved H3 10.8 mm to (200.0, 48.0)
- moved C30 10.2 mm to (180.3, 83.2)
- moved J3 7.62 mm to (192.8, 107.0)
- moved H2 5.06 mm to (115.0, 120.0)
- moved U6 4.37 mm to (180.6, 86.5), turned to 0 degrees
- moved SWBOOT1 2.59 mm to (142.8, 63.1), turned to 180 degrees
- moved J4 2.56 mm to (195.8, 85.2)
- moved R1 1.61 mm to (142.1, 69.2)
- moved U7 1.21 mm to (174.5, 84.9), turned to 180 degrees
- moved R3 0.45 mm to (182.2, 103.2)
- moved H1 0.35 mm to (115.0, 48.0)
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- renumbered C28 to C1, C18 to C16, C16 to C18, C30 to C19, C29 to C2, C31 to C20, C32 to C21, C35 to C22, C37 to C23, C38 to C24, C33 to C25, C34 to C26, C36 to C27, C5 to C28, C6 to C29, C20 to C3, C7 to C30, C8 to C31, C22 to C32, C24 to C33, C26 to C34, C23 to C35, C25 to C36, C27 to C37, C21 to C38, C19 to C4, C1 to C5, C2 to C6, C3 to C7, C4 to C8, D5 to D1, D1 to D2, D2 to D3, D3 to D4, H3 to H2, H2 to H3, J6 to J3, J1 to J4, J3 to J5, J4 to J6, J5 to J7, J9 to J8, J8 to J9, R4 to R10, R26 to R11, R10 to R12, R12 to R13, R11 to R15, R13 to R16, R15 to R17, R27 to R18, R28 to R19, R16 to R2, R5 to R20, R6 to R21, R17 to R3, R18 to R4, R19 to R5, R20 to R6, R3 to R7, R2 to R8, R22 to R9, U7 to U1, U3 to U2, U2 to U3, U1 to U7, U9 to U8
Connections:
- net /USB-UART/D_N renamed /USB-UART/D-
- net /USB-UART/D_P renamed /USB-UART/D+
- U2 pad 29: Extra_5 -> unconnected-(U2-PC3-Pad29)
- U2 pad 44: Extra_4 -> unconnected-(U2-PC4-Pad44)
- U2 pad 45: Extra_3 -> unconnected-(U2-PC5-Pad45)
Routing:
- net SPI2_NSS: track 0.00 -> 72.3 mm, vias 0 -> 1
- net I2C4_SCL: track 0.00 -> 62.3 mm, vias 0 -> 1
- net SPI2_SCK: track 0.00 -> 60.1 mm, vias 0 -> 1
- net I2C4_SDA: track 0.00 -> 59.8 mm, vias 0 -> 1
- net SPI2_MISO: track 0.00 -> 59.4 mm, vias 0 -> 1
- net SPI2_MOSI: track 0.00 -> 58.4 mm, vias 0 -> 1
- net USART2_RX: track 0.00 -> 56.0 mm, vias 0 -> 1
- net USART2_TX: track 0.00 -> 45.4 mm, vias 0 -> 2
- net VBUS: track 0.00 -> 32.8 mm, vias 0 -> 2
- net /MCU/USART1_RX: track 0.00 -> 17.7 mm, vias 0 -> 2
- net /ExtraPeriphs/SD_MISO: track 0.00 -> 17.6 mm, vias 0 -> 2
- net /ExtraPeriphs/SD_MOSI: track 0.00 -> 17.1 mm
- net /ExtraPeriphs/SD_SCK: track 0.00 -> 15.9 mm
- net /USB-UART/D-: track 10.4 -> 26.2 mm, vias 0 -> 2
- net /MCU/USART1_TX: track 0.00 -> 15.8 mm
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Other:
- board size 103.8 x 82.5 mm -> 91 x 78 mm

Commit message: Power Routing
Parts:
- moved J3 3.85 mm to (195.6, 104.3), turned to 90 degrees
- moved R9 2.82 mm to (181.2, 116.2), turned to 0 degrees
- moved C25 1.00 mm to (174.4, 98.0), turned to 90 degrees
- moved TP4 0.86 mm to (146.5, 110.3)
- moved C27 0.60 mm to (174.8, 115.7)
- moved ? 0.30 mm to (161.7, 109.4)
- moved ? 0.30 mm to (162.1, 109.9)
- moved ? 0.30 mm to (161.3, 109.9)
- moved ? 0.30 mm to (162.4, 109.4)
- moved ? 0.30 mm to (162.8, 109.9)
- moved ? 0.10 mm to (158.2, 107.4)
- moved C20 0.10 mm to (168.0, 113.8)
Routing:
- net +3.3V: track 38.0 -> 102.1 mm, vias 0 -> 2
- net V_Batt: track 0.00 -> 57.2 mm
- net VBUS: track 32.8 -> 65.3 mm, vias 2 -> 4
- net /LipoPower/Monitor_SDA: track 2.78 -> 29.8 mm, vias 0 -> 2
- net /LipoPower/Monitor_SCL: track 5.07 -> 30.6 mm, vias 0 -> 2
- net /LipoPower/Recharge_ST2: track 0.00 -> 22.1 mm, vias 0 -> 2
- net V_5V: track 5.37 -> 27.2 mm
- net /LipoPower/Recharge_PG: track 0.00 -> 21.6 mm, vias 0 -> 2
- net /LipoPower/Recharge_ST1: track 0.00 -> 18.9 mm, vias 0 -> 2
- net GND: track 56.0 -> 73.4 mm, vias 13 -> 20
- net /LipoPower/Monitor_GPOUT: track 0.00 -> 2.83 mm
- net Net-(U5-V_{DD}): track 0.00 -> 2.74 mm
- net Net-(U5-SRN): track 0.00 -> 2.66 mm
- net SPI2_MISO: track 59.4 -> 60.2 mm
- net SPI2_MOSI: track 58.4 -> 59.2 mm
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
Commit message: pushing
Parts:
- moved U6 2.51 mm to (180.8, 89.0)
Routing:
- net /USB-UART/D-: track 26.2 -> 0.00 mm, vias 2 -> 0
- net /USB-UART/D+: track 25.9 -> 0.00 mm
- net GND: track 73.4 -> 94.7 mm, vias 20 -> 31
- net V_Batt: track 57.2 -> 54.3 mm
- net Extra_3: track 44.2 -> 45.4 mm
- net /ExtraPeriphs/SD_SCK: track 15.9 -> 16.4 mm
- added copper zone on In1.Cu, net GND
- added copper zone on In2.Cu, net GND
- removed copper zone on B.Cu, net GND
Other:
- copper layers 2 -> 4

Commit message: pushing
Parts:
- removed U6: NUP2202, Package_TO_SOT_SMD:SOT-363_SC-70-6
- added C40: C_Small, Capacitor_SMD:C_0805_2012Metric_Pad1.18x1.45mm_HandSolder, F.Cu at (162.8, 66.5)
- added R22: R_Small, Resistor_SMD:R_0805_2012Metric_Pad1.20x1.40mm_HandSolder, F.Cu at (140.2, 104.8)
- added TP21: ~, TestPoint:TestPoint_Pad_1.0x1.0mm, F.Cu at (60.9, 88.3)
- added TP22: ~, TestPoint:TestPoint_Pad_1.0x1.0mm, F.Cu at (60.9, 91.3)
- added TP23: ~, TestPoint:TestPoint_Pad_1.0x1.0mm, F.Cu at (60.9, 94.4)
- added TP24: ~, TestPoint:TestPoint_Pad_1.0x1.0mm, F.Cu at (60.9, 97.5)
- added TP26: ~, TestPoint:TestPoint_Pad_1.0x1.0mm, F.Cu at (60.9, 100.5)
- added U9: USBLC6-2SC6, Package_TO_SOT_SMD:SOT-23-6, F.Cu at (182.1, 86.0)
- moved TP5 67.1 mm to (66.0, 85.0)
- moved TP6 67.1 mm to (66.0, 89.0)
- moved TP7 67.1 mm to (70.0, 85.0)
- moved TP8 67.1 mm to (70.0, 89.0)
- moved U1 3.75 mm to (139.5, 111.5)
- moved R18 2.87 mm to (167.5, 68.8)
- moved C2 0.50 mm to (138.0, 94.5)
Connections:
- net /USB-UART/D+ renamed /USB-UART/USB_D+
- net /USB-UART/D- renamed /USB-UART/USB_D-
Routing:
- net +3.3V: track 102.1 -> 74.4 mm, vias 2 -> 17
- net GND: track 94.7 -> 116.2 mm, vias 31 -> 43
- net /USB-UART/USB_D+: track 0.00 -> 18.9 mm
- net /USB-UART/USB_D-: track 0.00 -> 16.7 mm
- net VBUS: track 65.3 -> 54.6 mm
- net Net-(U7-VDD): track 0.00 -> 4.96 mm
- net NRST: track 15.5 -> 19.1 mm
- net Net-(U8-4A): track 3.30 -> 6.04 mm
- net V_Batt: track 54.3 -> 51.9 mm
- net SPI2_MOSI: track 59.2 -> 60.1 mm
- net SPI2_MISO: track 60.2 -> 60.9 mm
- added copper zone on B.Cu, net +3.3V

Commit message: pushing
Parts:
- moved H4 1.83 mm to (198.2, 119.7)
- moved H3 1.80 mm to (198.2, 48.0)
- moved H2 0.20 mm to (115.0, 119.8)
Routing:
- net GND: track 116.2 -> 120.4 mm, vias 43 -> 46
Other:
- board size 91 x 78 mm -> 89.2 x 77.8 mm
Changed lines of the file:
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@@
 		(tags "capacitor handsolder")
 		(property "Reference" "C29"
-			(at 3.4625 -0.25 0)
+			(at 3.4625 -0.5 0)
 			(layer "F.SilkS")
 			(effects
@@
 		(tags "capacitor handsolder")
 		(property "Reference" "C31"
-			(at 3.4625 0 0)
+			(at -0.7875 2 0)
 			(layer "F.SilkS")
 			(effects
@@
 	(footprint "MountingHole:MountingHole_2.1mm"
 		(layer "F.Cu")
-		(at 115 120)
+		(at 115 119.8)
 		(descr "Mounting Hole 2.1mm, no annular")
 		(tags "mounting hole 2.1mm no annular")
@@
 	(footprint "MountingHole:MountingHole_2.1mm"
 		(layer "F.Cu")
-		(at 200 120)
+		(at 198.2 119.65)
 		(descr "Mounting Hole 2.1mm, no annular")
 		(tags "mounting hole 2.1mm no annular")
@@
 		)
 		(pad "" np_thru_hole circle
-			(at 0 0)
+			(at 0 0.05)
 			(size 2.1 2.1)
 			(drill 2.1)
-			(layers "*.Cu" "*.Mask")
+			(layers "F&B.Cu" "*.Mask")
 		)
 	)
@@
 	(footprint "MountingHole:MountingHole_2.1mm"
 		(layer "F.Cu")
-		(at 200 48)
+		(at 198.2 48)
 		(descr "Mounting Hole 2.1mm, no annular")
 		(tags "mounting hole 2.1mm no annular")
@@
 		)
 	)
-	(gr_line
-		(start 115 45)
-		(end 200 45)
+	(gr_arc
+		(start 198.22 45.000001)
+		(mid 200.328426 45.885716)
+		(end 201.200066 48)
 		(stroke
 			(width 0.05)
@@
 	)
 	(gr_line
-		(start 112 120)
-		(end 112 48)
+		(start 198.2 122.8)
+		(end 114.99976 122.8)
 		(stroke
 			(width 0.05)
@@
 	)
 	(gr_line
-		(start 200 122.75)
-		(end 115 123)
+		(start 112 119.8)
+		(end 112 48)
 		(stroke
 			(width 0.05)
@@
 		(layer "Edge.Cuts")
 	)
-	(gr_arc
-		(start 200 45)
-		(mid 202.12132 45.87868)
-		(end 203 48)
+	(gr_line
+		(start 201.2 80.25)
+		(end 201.2 48)
 		(stroke
 			(width 0.05)
@@
 	)
 	(gr_line
-		(start 202.75 120)
-		(end 203 48)
+		(start 201.2 80.25)
+		(end 201.2 119.8)
 		(stroke
 			(width 0.05)
@@
 	)
 	(gr_arc
-		(start 115 123)
-		(mid 112.87868 122.12132)
-		(end 112 120)
+		(start 201.2 119.8)
+		(mid 200.32132 121.92132)
+		(end 198.2 122.8)
 		(stroke
 			(width 0.05)
@@
 	)
 	(gr_arc
-		(start 202.75 120)
-		(mid 201.944544 121.944544)
-		(end 200 122.75)
+		(start 114.99976 122.8)
+		(mid 112.878595 121.921235)
+		(end 112 119.8)
+		(stroke
+			(width 0.05)
+			(type default)
+		)
+		(layer "Edge.Cuts")
+	)
+	(gr_line
+		(start 198.22 45)
+		(end 115 45)
 		(stroke
 			(width 0.05)
@@
 	)
 	(segment
+		(start 174 80.5)
+		(end 173.25 79.75)
+		(width 0.5)
+		(layer "F.Cu")
+		(net 15)
+	)
+	(segment
 		(start 161.50312 101.75)
 		(end 161.5 101.75)
@@
 	)
 	(segment
+		(start 174.675 80.5)
+		(end 174 80.5)
+		(width 0.5)
+		(layer "F.Cu")
+		(net 15)
+	)
+	(segment
 		(start 151.75 100.6625)
 		(end 151.75 99.5)
@@
 	)
 	(segment
+		(start 174.675 78.25)
+		(end 173.25 78.25)
+		(width 0.6)
+		(layer "F.Cu")
+		(net 15)
+	)
+	(segment
 		(start 156.75 100.6625)
 		(end 156.75 99.5)
@@
 	)
 	(segment
+		(start 183.275 86)
+		(end 184.266231 86)
+		(width 0.3)
+		(layer "F.Cu")
+		(net 15)
+	)
+	(segment
 		(start 166.4 116.3)
 		(end 167.9 116.3)
@@
 	)
 	(segment
+		(start 184.266231 86)
+		(end 184.282871 86.01664)
+		(width 0.3)
+		(layer "F.Cu")
+		(net 15)
+	)
+	(segment
 		(start 131.5 90.25)
 		(end 133 90.25)
@@
 	)
 	(via
+		(at 173.25 79.75)
+		(size 0.7)
+		(drill 0.3)
+		(layers "F.Cu" "B.Cu")
+		(net 15)
+	)
+	(via
 		(at 182.3 113.1)
 		(size 0.6)
@@
 	)
 	(via
+		(at 184.282871 86.01664)
+		(size 0.7)
+		(drill 0.3)
+		(layers "F.Cu" "B.Cu")
+		(net 15)
+	)
+	(via
 		(at 156.75 80.75)
 		(size 0.7)
@@
 	)
 	(via
+		(at 173.25 78.25)
+		(size 0.7)
+		(drill 0.3)
+		(layers "F.Cu" "B.Cu")
+		(net 15)
+	)
+	(via
 		(at 132.5 79)
 		(size 0.7)
@@
 	)
 	(segment
+		(start 178.25 71.664212)
+		(end 178.25 47)
+		(width 0.3)
+		(layer "B.Cu")
+		(net 65)
+	)
+	(segment
 		(start 161.030761 89.169239)
 		(end 166.75 83.45)
@@
 	)
 	(segment
-		(start 168.3 83.45)
-		(end 178.25 73.5)
+		(start 168.45 81.464212)
+		(end 178.25 71.664212)
 		(width 0.3)
 		(layer "B.Cu")
@@
 	)
 	(segment
-		(start 161.7 95.2)
-		(end 161.030761 94.530761)
+		(start 167.747057 83.45)
+		(end 168.45 82.747057)
 		(width 0.3)
 		(layer "B.Cu")
@@
 	)
 	(segment
-		(start 166.75 83.45)
-		(end 168.3 83.45)
+		(start 168.45 82.747057)
+		(end 168.45 81.464212)
 		(width 0.3)
 		(layer "B.Cu")
@@
 	)
 	(segment
-		(start 178.25 73.5)
-		(end 178.25 47)
+		(start 166.75 83.45)
+		(end 167.747057 83.45)
 		(width 0.3)
 		(layer "B.Cu")
@@
 	)
 	(segment
+		(start 161.7 95.2)
+		(end 161.030761 94.530761)
+		(width 0.3)
+		(layer "B.Cu")
+		(net 65)
+	)
+	(segment
 		(start 162.5 97.75)
 		(end 164.1625 97.75)
@@
 	(segment
 		(start 177.25 47)
-		(end 177.25 73.5)
+		(end 177.25 71.957106)
 		(width 0.3)
 		(layer "B.Cu")
@@
 	)
 	(segment
-		(start 160.530761 88.962132)
-		(end 160.530761 95.780761)
+		(start 167.53995 82.95)
+		(end 166.542893 82.95)
+		(width 0.3)
+		(layer "B.Cu")
+		(net 66)
+	)
+	(segment
+		(start 160.530761 95.780761)
+		(end 162.25 97.5)
 		(width 0.3)
 		(layer "B.Cu")
@@
 	)
 	(segment
-		(start 177.25 73.5)
-		(end 167.8 82.95)
+		(start 160.530761 88.962132)
+		(end 160.530761 95.780761)
 		(width 0.3)
 		(layer "B.Cu")
@@
 	)
 	(segment
-		(start 167.8 82.95)
-		(end 166.542893 82.95)
+		(start 167.95 81.257106)
+		(end 167.95 82.53995)
 		(width 0.3)
 		(layer "B.Cu")
@@
 	)
 	(segment
-		(start 160.530761 95.780761)
-		(end 162.25 97.5)
+		(start 167.95 82.53995)
+		(end 167.53995 82.95)
+		(width 0.3)
+		(layer "B.Cu")
+		(net 66)
+	)
+	(segment
+		(start 177.25 71.957106)
+		(end 167.95 81.257106)
 		(width 0.3)
 		(layer "B.Cu")
