File: EInkDisplay-PCB/ECE477-SeniorDesign/ECE477-SeniorDesign.kicad_pcb (KiCad board)
At the start: 4 copper layers, 89.2 x 77.8 mm, 138 parts, among them J10 Conn_01x05_Pin, J11 Conn_01x05_Pin, J2 Conn_01x05_Pin, J3 Battery Connector, J4 USB_A, J5 JST Conn, J6 JST Conn, J7 JST Conn, J8 Micro_SD_Card_Det1, J9 JST Conn, U1 PTS526 SK15 SMTR2 LFS, U2 STM32L496ZGTxP, U3 MCP73871, U4 TPS63060, U5 BQ27441-G1, U7 CP2102-GMR, U8 74LVC125APW_118, U9 USBLC6-2SC6, Y1 Y1

Commit message: pushing
Parts:
- removed C25: 4.7 uF, Capacitor_SMD:C_0805_2012Metric_Pad1.18x1.45mm_HandSolder
- removed the J3 at (195.6, 104.3)
- removed J5: JST Conn, PCB_Lib:JST Conn
- removed the R2 at (184.3, 102.8)
- removed R3, R4: 15K, Resistor_SMD:R_0805_2012Metric_Pad1.20x1.40mm_HandSolder
- removed R5: 1.2M, Resistor_SMD:R_0805_2012Metric_Pad1.20x1.40mm_HandSolder
- removed U3: MCP73871, Package_DFN_QFN:QFN-20-1EP_4x4mm_P0.5mm_EP2.5x2.5mm
- added C28: 4.7 uF, Capacitor_SMD:C_0805_2012Metric_Pad1.18x1.45mm_HandSolder, F.Cu at (173.8, 98.9)
- added C29: 4.7 uF, Capacitor_SMD:C_0805_2012Metric_Pad1.18x1.45mm_HandSolder, F.Cu at (178.2, 95.5)
- added C30: 4.7 uF, Capacitor_SMD:C_0805_2012Metric_Pad1.18x1.45mm_HandSolder, F.Cu at (183.2, 98.9)
- added J8: JST Conn, PCB_Lib:JST Conn, F.Cu at (116.9, 75.4)
- added R10: 470, Resistor_SMD:R_0805_2012Metric_Pad1.20x1.40mm_HandSolder, F.Cu at (213.2, 100.5)
- added R12: 470, Resistor_SMD:R_0805_2012Metric_Pad1.20x1.40mm_HandSolder, F.Cu at (222.3, 95.4)
- added R13: 470, Resistor_SMD:R_0805_2012Metric_Pad1.20x1.40mm_HandSolder, F.Cu at (222.3, 98.4)
- added R14: 10K, Resistor_SMD:R_0805_2012Metric_Pad1.20x1.40mm_HandSolder, F.Cu at (222.3, 101.3)
- added R16: 15k, Resistor_SMD:R_0805_2012Metric_Pad1.20x1.40mm_HandSolder, F.Cu at (222.3, 104.3)
- added R17: 1k, Resistor_SMD:R_0805_2012Metric_Pad1.20x1.40mm_HandSolder, F.Cu at (222.3, 107.2)
- added R18: 15k, Resistor_SMD:R_0805_2012Metric_Pad1.20x1.40mm_HandSolder, F.Cu at (222.3, 110.2)
- added R6: 1.2M, Resistor_SMD:R_0805_2012Metric_Pad1.20x1.40mm_HandSolder, F.Cu at (149.1, 114.9)
- added U6: MCP73871-2CCI/ML, PCB_Lib:MCP73871, F.Cu at (178.5, 100.4)
- J6: value JST Conn -> Battery Connector
- moved J6 82.8 mm to (195.2, 102.4), turned to 90 degrees
- moved J9 12.9 mm to (116.9, 86.3)
- moved J10 12.9 mm to (116.8, 99.2)
- renumbered C3 to C1, C1 to C2, C2 to C3, C28 to C31, C29 to C32, C30 to C33, C31 to C34, C32 to C35, C33 to C36, C34 to C37, C35 to C38, C36 to C39, C37 to C40, C40 to C41, C38 to C42, C39 to C43, D1 to D4, D2 to D5, D3 to D6, D4 to D7, J7 to J10, J8 to J11, J10 to J3, J11 to J4, J4 to J7, R22 to R1, R9 to R11, R10 to R15, R11 to R19, R1 to R2, R12 to R20, R13 to R21, R14 to R22, R15 to R23, R16 to R24, R17 to R25, R18 to R26, R19 to R27, R20 to R28, R21 to R29, R6 to R7, R7 to R8, R8 to R9, TP9 to TP10, TP10 to TP11, TP11 to TP12, TP12 to TP13, TP25 to TP21, TP21 to TP22, TP22 to TP23, TP23 to TP24, TP24 to TP25, TP13 to TP9, U9 to U7, U7 to U8, U8 to U9
Connections:
- D5 pad 2: Net-(D2-A) -> Net-(D5-A)
- D7 pad 2: Net-(D4-A) (its old number) -> Net-(D7-A)
- J6 pad 1: +3.3V -> V_Batt
- J6 pad 2: Net-(D2-A) -> GND
- J9 pad 2: Net-(D4-A) (its old number) -> Net-(D5-A)
- R21 pad 1: Net-(D2-A) -> Net-(D5-A)
- R28 pad 1: Net-(D4-A) (its old number) -> Net-(D7-A)
Routing:
- net V_Batt: track 51.9 -> 26.6 mm
- net VBUS: track 54.6 -> 30.7 mm, vias 4 -> 2
- net V_5V: track 27.2 -> 8.52 mm
- net Net-(D5-A): track 0.00 -> 9.08 mm
- net Net-(D2-A): track 9.08 -> 0.00 mm
- net Net-(D7-A): track 0.00 -> 6.08 mm
- net Net-(D4-A) (its old number): track 6.08 -> 0.00 mm
- net GND: track 120.4 -> 115.1 mm
- net Net-(U3-PROG1): track 4.39 -> 0.00 mm
- net Net-(U5-V_{DD}): track 2.74 -> 0.00 mm
- net Net-(U3-PROG3): track 2.26 -> 0.00 mm
- net Net-(U3-THERM): track 1.81 -> 0.00 mm
- net +3.3V: track 74.4 -> 72.8 mm, vias 17 -> 18
- added copper zone on F.Cu, net V_5V
- added copper zone on F.Cu, net V_Batt
- removed copper zone on F.Cu, net GND

Commit message: pusj
Parts:
- removed R10, R12, R13: 470, Resistor_SMD:R_0805_2012Metric_Pad1.20x1.40mm_HandSolder
- added C25: 1uF, Capacitor_SMD:C_0805_2012Metric_Pad1.18x1.45mm_HandSolder, F.Cu at (177.2, 117.0)
- added J12: JST Conn, PCB_Lib:JST Conn, F.Cu at (116.9, 99.2)
- added R3: 1.8M, Resistor_SMD:R_0805_2012Metric_Pad1.20x1.40mm_HandSolder, F.Cu at (185.0, 110.6)
- moved R14 48.5 mm to (173.8, 102.2)
- moved R16 46.0 mm to (176.3, 105.1), turned to 90 degrees
- moved R18 40.2 mm to (182.6, 104.0), turned to 90 degrees
- moved R17 38.9 mm to (184.0, 100.9)
- moved J10 11.9 mm to (116.8, 87.3)
- moved J8 10.4 mm to (116.7, 65.0)
- moved J9 10.1 mm to (116.7, 76.2)
- moved J6 8.27 mm to (196.3, 110.6)
- moved R11 4.67 mm to (185.8, 115.4), turned to -90 degrees
- moved C27 1.13 mm to (174.2, 114.8), turned to 180 degrees
- moved TP1 0.60 mm to (169.6, 84.5)
Connections:
- J6 pad 1: V_Batt -> BATTERY_IN
- R11 pad 1: V_Batt -> BATTERY_IN
- R11 pad 2: Net-(U5-SRN) -> V_Batt
- U5 pad 10: GND -> Net-(U5-BIN)
- U5 pad 6: V_Batt -> BATTERY_IN
- U5 pad 7: Net-(U5-SRN) -> V_Batt
- U5 pad 8: V_Batt -> BATTERY_IN
Routing:
- net /LipoPower/Monitor_GPOUT: track 2.83 -> 32.3 mm
- net V_Batt: track 26.6 -> 0.00 mm
- net GND: track 115.1 -> 122.3 mm, vias 46 -> 53
- net +3.3V: track 72.8 -> 78.0 mm, vias 18 -> 22
- net Net-(U5-BIN): track 0.00 -> 4.61 mm
- net /LipoPower/Monitor_SCL: track 30.6 -> 27.4 mm
- net V_5V: track 8.52 -> 5.37 mm
- net Net-(U5-SRN): track 2.66 -> 0.00 mm
- net Net-(U5-V_{DD}): track 0.00 -> 2.38 mm
- net BATTERY_IN: track 0.00 -> 2.26 mm
- net /MCU/USART1_RX: track 17.7 -> 16.0 mm
- net /LipoPower/Recharge_ST2: track 21.7 -> 23.3 mm
- net /LipoPower/Recharge_PG: track 21.6 -> 22.8 mm
- removed copper zone on F.Cu, net V_5V
- removed copper zone on F.Cu, net V_Batt

Commit message: done
Parts:
- removed the ? at (162.5, 113.8)
- removed the ? at (161.3, 109.9)
- removed the ? at (162.5, 114.5)
- removed the ? at (161.3, 115.0)
- removed the ? at (161.7, 109.4)
- removed the ? at (162.8, 115.0)
- removed the ? at (161.7, 113.8)
- removed the ? at (162.1, 109.9)
- removed the ? at (161.7, 114.5)
- removed the ? at (162.1, 115.0)
- removed the ? at (162.4, 109.4)
- removed the ? at (162.8, 109.9)
- removed TP11, TP12, TP13, TP16, TP17, TP18, TP19, TP20, TP25, TP26: ~, TestPoint:TestPoint_Pad_1.0x1.0mm
- removed TP14: BOOT0, TestPoint:TestPoint_Pad_1.0x1.0mm
- removed the TP21 at (68.0, 71.5)
- removed the TP22 at (60.9, 88.3)
- removed the TP23 at (60.9, 91.3)
- removed the TP24 at (60.9, 94.4)
- removed TP3: E_MOSI, TestPoint:TestPoint_Pad_1.0x1.0mm
- removed TP4: E_NSS, TestPoint:TestPoint_Pad_1.0x1.0mm
- removed TP5: E_RST, TestPoint:TestPoint_Pad_1.0x1.0mm
- removed TP6: E_SCK, TestPoint:TestPoint_Pad_1.0x1.0mm
- removed TP7: E_D/C, TestPoint:TestPoint_Pad_1.0x1.0mm
- removed TP8: E_Busy, TestPoint:TestPoint_Pad_1.0x1.0mm
- removed TP9: NSRT, TestPoint:TestPoint_Pad_1.0x1.0mm
- added EinkDispCon1: ~, Connector_PinHeader_1.00mm:PinHeader_1x08_P1.00mm_Vertical, F.Cu at (138.1, 120.8)
- U4: footprint Package_SON:Texas_S-PWSON-N10_ThermalVias -> PCB_Lib:DSC0010E
- moved R6 4.33 mm to (151.9, 118.2)
- moved R11 1.10 mm to (184.7, 115.5)
- moved U5 0.14 mm to (179.3, 113.4)
Routing:
- net /MCU/Eink_D/C: track 0.00 -> 51.5 mm, vias 0 -> 1
- net /MCU/Eink_RST: track 0.00 -> 48.2 mm, vias 0 -> 1
- net V_Batt: track 0.00 -> 46.8 mm
- net VBUS: track 30.7 -> 61.0 mm
- net /MCU/SPI1_SCK: track 0.00 -> 28.3 mm, vias 0 -> 1
- net /MCU/SPI1_NSS: track 0.00 -> 24.9 mm, vias 0 -> 1
- net /MCU/SPI1_MOSI: track 0.00 -> 23.8 mm, vias 0 -> 2
- net /MCU/Eink_Busy: track 0.00 -> 21.3 mm, vias 0 -> 2
- net BATTERY_IN: track 2.26 -> 14.7 mm
- net GND: track 122.3 -> 129.2 mm, vias 53 -> 57
- net Net-(U6-PROG3): track 0.00 -> 3.25 mm
- net Net-(U6-THERM): track 0.00 -> 2.83 mm
- net Net-(U6-PROG1): track 0.00 -> 2.81 mm
- net Net-(U6-PROG2): track 0.00 -> 2.59 mm
- net V_5V: track 5.37 -> 7.39 mm
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
Commit message: push
Parts:
- removed the ? at (158.2, 107.4)
- removed J11: Micro_SD_Card_Det1, PCB_Lib:SD_Reader
- removed TP1: UART_TX, TestPoint:TestPoint_Pad_1.0x1.0mm
- removed TP10, TP15, TP21, TP22, TP23, TP24: ~, TestPoint:TestPoint_Pad_1.0x1.0mm
- removed TP2: UART_RX, TestPoint:TestPoint_Pad_1.0x1.0mm
- removed TP27: VBUS, TestPoint:TestPoint_Pad_1.0x1.0mm
- added CARD1: ~, PCB_Lib:SD_reader_comp, F.Cu at (157.7, 55.2)
- moved R14 9.72 mm to (179.6, 94.4), turned to -90 degrees
- moved R16 9.51 mm to (176.7, 95.6), turned to 0 degrees
- moved C28 9.51 mm to (182.6, 95.3), turned to 0 degrees
- moved R8 9.32 mm to (178.2, 118.3), turned to -90 degrees
- moved D4 8.31 mm to (132.0, 60.0), turned to 180 degrees
- moved R6 7.96 mm to (155.3, 111.0)
- moved R3 7.80 mm to (177.3, 109.4), turned to -90 degrees
- moved C29 7.56 mm to (184.9, 98.9), turned to 0 degrees
- moved C27 7.52 mm to (180.4, 119.0), turned to -90 degrees
- moved R11 6.77 mm to (180.3, 110.4), turned to 0 degrees
- moved R15 6.13 mm to (175.3, 112.3)
- moved R18 6.04 mm to (176.7, 102.7), turned to 0 degrees
- moved J6 5.93 mm to (196.9, 104.7)
- moved R9 5.87 mm to (175.3, 116.0), turned to 180 degrees
- moved SWBOOT1 5.80 mm to (139.3, 67.8), turned to -90 degrees
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Connections:
- EinkDispCon1 pad 1: +3.3V -> /MCU/SPI1_NSS
- EinkDispCon1 pad 2: GND -> /MCU/SPI1_SCK
- EinkDispCon1 pad 3: /MCU/SPI1_MOSI -> /MCU/Eink_Busy
- EinkDispCon1 pad 4: /MCU/SPI1_SCK -> /MCU/SPI1_MOSI
- EinkDispCon1 pad 5: /MCU/SPI1_NSS -> /MCU/Eink_D/C
- EinkDispCon1 pad 6: /MCU/Eink_D/C -> /MCU/Eink_RST
- EinkDispCon1 pad 7: /MCU/Eink_RST -> GND
- EinkDispCon1 pad 8: /MCU/Eink_Busy -> +3.3V
- R26 pad 2: DO_LLC -> DO_LLS
- U2 pad 103: /MCU/Eink_D/C -> unconnected-(U2-PA11-Pad103)
- U2 pad 104: /MCU/Eink_RST -> unconnected-(U2-PA12-Pad104)
- U2 pad 44: unconnected-(U2-PC4-Pad44) -> /MCU/Eink_D/C
- U2 pad 45: unconnected-(U2-PC5-Pad45) -> /MCU/Eink_RST
- U9 pad 8: CS_LLC -> CS_LLS
Routing:
- net SPI2_NSS: track 72.3 -> 0.00 mm, vias 1 -> 0
- net I2C4_SCL: track 62.4 -> 0.00 mm, vias 1 -> 0
- net SPI2_SCK: track 60.8 -> 0.00 mm, vias 1 -> 0
- net SPI2_MISO: track 60.7 -> 0.00 mm, vias 1 -> 0
- net I2C4_SDA: track 59.8 -> 0.00 mm, vias 1 -> 0
- net SPI2_MOSI: track 59.8 -> 0.00 mm, vias 1 -> 0
- net GND: track 129.2 -> 71.2 mm, vias 57 -> 30
- net USART2_RX: track 56.0 -> 0.00 mm, vias 1 -> 0
- net Extra_2: track 51.7 -> 0.00 mm
- net /MCU/Eink_D/C: track 51.5 -> 0.00 mm, vias 1 -> 0
- net /MCU/Eink_RST: track 48.2 -> 0.00 mm, vias 1 -> 0
- net V_Batt: track 46.8 -> 0.00 mm
- net Extra_3: track 45.4 -> 0.00 mm, vias 1 -> 0
- net USART2_TX: track 45.4 -> 0.00 mm, vias 2 -> 0
- net Extra_1: track 42.5 -> 0.00 mm
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
Commit message: pusbh
Parts:
- moved D7 1.10 mm to (132.0, 96.4)
- moved C42 1.00 mm to (130.6, 102.0)
- moved C43 1.00 mm to (132.8, 102.1)
- moved R29 1.00 mm to (131.6, 99.0)
- moved R28 0.43 mm to (124.7, 101.1)
Routing:
- net USART2_TX: track 0.00 -> 46.4 mm, vias 0 -> 1
- net USART2_RX: track 0.00 -> 42.1 mm, vias 0 -> 1
- net Extra_2: track 0.00 -> 38.9 mm, vias 0 -> 1
- net Extra_1: track 0.00 -> 38.1 mm, vias 0 -> 1
- net Extra_5: track 0.00 -> 38.0 mm, vias 0 -> 1
- net Extra_4: track 0.00 -> 37.9 mm, vias 0 -> 1
- net Extra_3: track 0.00 -> 37.6 mm, vias 0 -> 1
- net /ExtraPeriphs/switch: track 0.00 -> 25.0 mm
- net /ExtraPeriphs/button1: track 0.00 -> 23.5 mm
- net /ExtraPeriphs/button3: track 0.00 -> 17.1 mm
- net /ExtraPeriphs/button2: track 0.00 -> 16.0 mm
- net GND: track 71.2 -> 87.2 mm, vias 30 -> 40
- net NRST: track 5.01 -> 18.8 mm, vias 0 -> 2
- net Net-(U2-PH3): track 0.00 -> 12.8 mm
- net +3.3V: track 55.4 -> 67.9 mm, vias 16 -> 21
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
Commit message: Regulator footprint and sch update
Parts:
- removed U4: TPS63060, PCB_Lib:DSC0010E
- added R4: 91k, Resistor_SMD:R_0805_2012Metric_Pad1.20x1.40mm_HandSolder, F.Cu at (127.6, 110.5)
- added U10: TPS63802DLA, Project_PCB_Library:TPS63802DLR, F.Cu at (125.5, 119.6)
- C20: value 10uF -> 22uF
- L1: value 1uH -> 470nH; footprint Inductor_SMD:L_1008_2520Metric_Pad1.43x2.20mm_HandSolder -> Project_PCB_Library:IND_XFL4015_COC-L
- R6: value 1.2M -> 100k
- R7: value 200k -> 511k
- moved C19 40.1 mm to (126.3, 119.9), turned to 180 degrees
- moved L1 34.8 mm to (127.2, 116.9), turned to -90 degrees
- moved C20 21.0 mm to (147.2, 116.7)
Connections:
- C20 pad 1: V_5V -> +3.3V
- R6 pad 2: Net-(U4-FB) -> Net-(U10-PG)
- R7 pad 1: Net-(U4-FB) -> +3.3V
- R7 pad 2: GND -> Net-(U10-FB)

Commit message: push
Parts:
- added J1: Conn_01x05_Pin, Connector_PinHeader_1.00mm:PinHeader_1x05_P1.00mm_Vertical, F.Cu at (184.2, 47.0)
- C2: value 4pF -> 6pF
- C3: value 4pF -> 6pf
- Y1: value Y1 -> CM9V-T1A-32.768KHZ-7PF-100PPM-TA-QC; footprint PCB_Lib:XTAL_ABS04W-32.768KHZ-4-D2-T5 -> PCB_Lib:CM9V-T1A-32.768KHZ-7PF-100PPM-TA-QC
- moved C20 9.59 mm to (156.6, 118.5)
- moved R4 8.35 mm to (121.5, 116.2)
- moved U7 0.94 mm to (181.2, 86.0)
- moved Y1 0.38 mm to (135.8, 92.2), turned to -90 degrees
Connections:
- J3 pad 3: SPI2_MOSI -> SPI2_SCK
- J3 pad 5: SPI2_SCK -> SPI2_MOSI
- J4 pad 2: USART2_RX -> USART2_TX
- J4 pad 3: USART2_TX -> USART2_RX
- U2 pad 114: unconnected-(U2-PD0-Pad114) -> SPI2_NSS
- U2 pad 115: unconnected-(U2-PD1-Pad115) -> SPI2_SCK
- U2 pad 117: unconnected-(U2-PD3-Pad117) -> SPI2_MISO
- U2 pad 118: unconnected-(U2-PD4-Pad118) -> SPI2_MOSI
- U2 pad 139: SPI2_NSS -> unconnected-(U2-PB9-Pad139)
- U2 pad 69: SPI2_SCK -> unconnected-(U2-PB10-Pad69)
- U2 pad 75: SPI2_MISO -> unconnected-(U2-PB14-Pad75)
- U2 pad 76: SPI2_MOSI -> unconnected-(U2-PB15-Pad76)
- Y1 pad 2: GND -> Net-(U2-PH1)
Routing:
- net NRST: track 18.8 -> 88.6 mm, vias 2 -> 3
- net I2C4_SCL: track 0.00 -> 52.2 mm, vias 0 -> 1
- net I2C4_SDA: track 0.00 -> 51.2 mm, vias 0 -> 1
- net SWDIO: track 0.00 -> 47.2 mm, vias 0 -> 2
- net SPI2_MISO: track 0.00 -> 46.5 mm, vias 0 -> 1
- net SPI2_SCK: track 0.00 -> 46.1 mm, vias 0 -> 1
- net SWCLK: track 0.00 -> 45.7 mm, vias 0 -> 2
- net SPI2_NSS: track 1.98 -> 45.0 mm
- net SPI2_MOSI: track 0.00 -> 42.7 mm, vias 0 -> 1
- net /MCU/SPI1_SCK: track 0.00 -> 31.7 mm, vias 0 -> 2
- net /MCU/SPI1_NSS: track 0.00 -> 27.8 mm, vias 0 -> 1
- net /MCU/Eink_RST: track 0.00 -> 23.6 mm, vias 0 -> 1
- net /MCU/Eink_Busy: track 0.00 -> 22.7 mm, vias 0 -> 1
- net /MCU/Eink_D/C: track 0.00 -> 22.5 mm, vias 0 -> 1
- net /MCU/SPI1_MOSI: track 0.00 -> 22.1 mm, vias 0 -> 1
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
Commit message: changes
Parts:
- removed ? (x2): , 
- removed C21: 0.1uF, Capacitor_SMD:C_0805_2012Metric_Pad1.18x1.45mm_HandSolder
- removed C22, C23, C24: 22uF, Capacitor_SMD:C_0805_2012Metric_Pad1.18x1.45mm_HandSolder
- removed C26: 10pF, Capacitor_SMD:C_0805_2012Metric_Pad1.18x1.45mm_HandSolder
- moved C19 36.8 mm to (162.2, 111.7)
- moved U10 36.2 mm to (161.7, 118.1)
- moved R4 36.2 mm to (157.5, 112.7), turned to 90 degrees
- moved L1 36.1 mm to (163.3, 115.4)
- moved R7 7.82 mm to (157.5, 116.5), turned to 90 degrees
- moved C20 6.02 mm to (162.6, 119.0), turned to 180 degrees
- moved R6 5.50 mm to (155.5, 116.5), turned to 90 degrees
Routing:
- net GND: track 92.1 -> 99.3 mm, vias 42 -> 46
- net Net-(U10-FB): track 0.00 -> 6.66 mm
- net Net-(U10-L2): track 0.00 -> 5.12 mm
- net Net-(U10-L1): track 0.00 -> 4.94 mm
- net +3.3V: track 72.5 -> 76.3 mm
- net V_5V: track 0.00 -> 2.84 mm
- added copper zone on F.Cu, net +3.3V
- added copper zone on F.Cu, net V_5V
