File: EInkDisplay-PCB/ECE477-SeniorDesign/ECE477-SeniorDesign.kicad_sch (KiCad schematic)
At the start: 13 parts

Commit message: whole lotta changes
Parts:
- H1, H2, H3, H4: footprint (none) -> MountingHole:MountingHole_2.1mm
Other:
- sheet MCU ports: added SPI3_MISO, SPI3_MOSI, SPI3_NSS, SPI3_SCK; removed SPI2_MISO, SPI2_MOSI, SPI2_NSS, SPI2_SCK
Changed lines of the file:
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@@
 			)
 		)
-		(property "Footprint" ""
+		(property "Footprint" "MountingHole:MountingHole_2.1mm"
 			(at 209.55 48.26 0)
 			(effects
@@
 			)
 		)
-		(property "Footprint" ""
+		(property "Footprint" "MountingHole:MountingHole_2.1mm"
 			(at 209.55 39.37 0)
 			(effects
@@
 			)
 		)
-		(property "Footprint" ""
+		(property "Footprint" "MountingHole:MountingHole_2.1mm"
 			(at 231.14 48.26 0)
 			(effects
@@
 			)
 		)
-		(property "Footprint" ""
+		(property "Footprint" "MountingHole:MountingHole_2.1mm"
 			(at 231.14 39.37 0)
 			(effects
@@
 			)
 		)
-		(pin "SPI2_NSS" input
-			(at 138.43 86.36 90)
-			(effects
-				(font
-					(size 1.27 1.27)
-				)
-				(justify right)
-			)
-		)
-		(pin "SPI2_SCK" input
-			(at 130.81 86.36 90)
-			(effects
-				(font
-					(size 1.27 1.27)
-				)
-				(justify right)
-			)
-		)
-		(pin "SPI2_MISO" input
-			(at 135.89 86.36 90)
-			(effects
-				(font
-					(size 1.27 1.27)
-				)
-				(justify right)
-			)
-		)
-		(pin "SPI2_MOSI" input
-			(at 133.35 86.36 90)
-			(effects
-				(font
-					(size 1.27 1.27)
-				)
-				(justify right)
-			)
-		)
 		(pin "SPI1_NSS" input
 			(at 182.88 124.46 0)
@@
 			)
 		)
+		(pin "I2C2_SDA" input
+			(at 116.84 120.65 180)
+			(effects
+				(font
+					(size 1.27 1.27)
+				)
+				(justify left)
+			)
+		)
+		(pin "I2C2_SCL" input
+			(at 116.84 118.11 180)
+			(effects
+				(font
+					(size 1.27 1.27)
+				)
+				(justify left)
+			)
+		)
+		(pin "GPIO_4" input
+			(at 116.84 129.54 180)
+			(effects
+				(font
+					(size 1.27 1.27)
+				)
+				(justify left)
+			)
+		)
+		(pin "GPIO_3" input
+			(at 116.84 123.19 180)
+			(effects
+				(font
+					(size 1.27 1.27)
+				)
+				(justify left)
+			)
+		)
+		(pin "GPIO_5" input
+			(at 116.84 132.08 180)
+			(effects
+				(font
+					(size 1.27 1.27)
+				)
+				(justify left)
+			)
+		)
+		(pin "GPIO_6" input
+			(at 116.84 134.62 180)
+			(effects
+				(font
+					(size 1.27 1.27)
+				)
+				(justify left)
+			)
+		)
+		(pin "SPI3_MISO" input
+			(at 135.89 86.36 90)
+			(effects
+				(font
+					(size 1.27 1.27)
+				)
+				(justify right)
+			)
+		)
+		(pin "SPI3_MOSI" input
+			(at 133.35 86.36 90)
+			(effects
+				(font
+					(size 1.27 1.27)
+				)
+				(justify right)
+			)
+		)
+		(pin "SPI3_SCK" input
+			(at 130.81 86.36 90)
+			(effects
+				(font
+					(size 1.27 1.27)
+				)
+				(justify right)
+			)
+		)
+		(pin "SPI3_NSS" input
+			(at 138.43 86.36 90)
+			(effects
+				(font
+					(size 1.27 1.27)
+				)
+				(justify right)
+			)
+		)
+		(pin "button2" input
+			(at 153.67 86.36 90)
+			(effects
+				(font
+					(size 1.27 1.27)
+				)
+				(justify right)
+			)
+		)
 		(pin "button1" input
 			(at 156.21 86.36 90)
@@
 			)
 		)
-		(pin "button2" input
-			(at 153.67 86.36 90)
-			(effects
-				(font
-					(size 1.27 1.27)
-				)
-				(justify right)
-			)
-		)
 		(pin "button3" input
 			(at 151.13 86.36 90)
@@
 			)
 		)
-		(pin "I2C2_SDA" input
-			(at 116.84 120.65 180)
-			(effects
-				(font
-					(size 1.27 1.27)
-				)
-				(justify left)
-			)
-		)
-		(pin "I2C2_SCL" input
-			(at 116.84 118.11 180)
-			(effects
-				(font
-					(size 1.27 1.27)
-				)
-				(justify left)
-			)
-		)
-		(pin "GPIO_4" input
-			(at 116.84 129.54 180)
-			(effects
-				(font
-					(size 1.27 1.27)
-				)
-				(justify left)
-			)
-		)
-		(pin "GPIO_3" input
-			(at 116.84 123.19 180)
-			(effects
-				(font
-					(size 1.27 1.27)
-				)
-				(justify left)
-			)
-		)
-		(pin "GPIO_5" input
-			(at 116.84 132.08 180)
-			(effects
-				(font
-					(size 1.27 1.27)
-				)
-				(justify left)
-			)
-		)
-		(pin "GPIO_6" input
-			(at 116.84 134.62 180)
-			(effects
-				(font
-					(size 1.27 1.27)
-				)
-				(justify left)
-			)
-		)

Commit message: pushing
Parts:
- renumbered EinkDispCon2 to EinkDispCon1, H3 to H2, H2 to H3, TP12 to TP1, TP13 to TP2, TP6 to TP3, TP8 to TP4, TP10 to TP5, TP7 to TP6, TP9 to TP7, TP11 to TP8
Other:
- sheet ExtraPeriphs ports: added switch; removed none
- sheet MCU ports: added switch; removed none
Changed lines of the file:
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@@
+	(wire
+		(pts
+			(xy 158.75 69.85) (xy 158.75 86.36)
+		)
+		(stroke
+			(width 0)
+			(type default)
+		)
+	)
 	(wire
 		(pts
@@
 		(dnp no)
 		(fields_autoplaced yes)
-		(property "Reference" "TP13"
+		(property "Reference" "TP2"
 			(at 101.6 78.2319 0)
 			(effects
@@
 			(project "ECE477-SeniorDesign"
 				(path "/527ae649-08be-4368-9cf9-441ebba18eca"
-					(reference "TP13")
+					(reference "TP2")
 					(unit 1)
 				)
@@
 		(dnp no)
 		(fields_autoplaced yes)
-		(property "Reference" "TP12"
+		(property "Reference" "TP1"
 			(at 101.6 69.0879 0)
 			(effects
@@
 			(project "ECE477-SeniorDesign"
 				(path "/527ae649-08be-4368-9cf9-441ebba18eca"
-					(reference "TP12")
+					(reference "TP1")
 					(unit 1)
 				)
@@
 		(dnp no)
 		(fields_autoplaced yes)
-		(property "Reference" "H3"
+		(property "Reference" "H2"
 			(at 212.09 46.9899 0)
 			(effects
@@
 			(project "ECE477-SeniorDesign"
 				(path "/527ae649-08be-4368-9cf9-441ebba18eca"
-					(reference "H3")
+					(reference "H2")
 					(unit 1)
 				)
@@
 		(on_board yes)
 		(dnp no)
-		(property "Reference" "EinkDispCon2"
+		(property "Reference" "EinkDispCon1"
 			(at 237.236 136.398 0)
 			(effects
@@
 			(project "ECE477-SeniorDesign"
 				(path "/527ae649-08be-4368-9cf9-441ebba18eca"
-					(reference "EinkDispCon2")
+					(reference "EinkDispCon1")
 					(unit 1)
 				)
@@
 		(dnp no)
 		(fields_autoplaced yes)
-		(property "Reference" "TP7"
+		(property "Reference" "TP6"
 			(at 204.47 117.3479 0)
 			(effects
@@
 			(project "ECE477-SeniorDesign"
 				(path "/527ae649-08be-4368-9cf9-441ebba18eca"
-					(reference "TP7")
+					(reference "TP6")
 					(unit 1)
 				)
@@
 		(dnp no)
 		(fields_autoplaced yes)
-		(property "Reference" "#PWR012"
+		(property "Reference" "#PWR01"
 			(at 223.52 113.03 0)
 			(effects
@@
 			(project ""
 				(path "/527ae649-08be-4368-9cf9-441ebba18eca"
-					(reference "#PWR012")
+					(reference "#PWR01")
 					(unit 1)
 				)
@@
 		(dnp no)
 		(fields_autoplaced yes)
-		(property "Reference" "TP9"
+		(property "Reference" "TP7"
 			(at 204.47 122.4279 0)
 			(effects
@@
 			(project "ECE477-SeniorDesign"
 				(path "/527ae649-08be-4368-9cf9-441ebba18eca"
-					(reference "TP9")
+					(reference "TP7")
 					(unit 1)
 				)
@@
 		(dnp no)
 		(fields_autoplaced yes)
-		(property "Reference" "#PWR013"
+		(property "Reference" "#PWR02"
 			(at 217.17 116.84 0)
 			(effects
@@
 			(project ""
 				(path "/527ae649-08be-4368-9cf9-441ebba18eca"
-					(reference "#PWR013")
+					(reference "#PWR02")
 					(unit 1)
 				)
@@
 		(dnp no)
 		(fields_autoplaced yes)
-		(property "Reference" "TP10"
+		(property "Reference" "TP5"
 			(at 193.04 124.9679 0)
 			(effects
@@
 			(project "ECE477-SeniorDesign"
 				(path "/527ae649-08be-4368-9cf9-441ebba18eca"
-					(reference "TP10")
+					(reference "TP5")
 					(unit 1)
 				)
@@
 		(dnp no)
 		(fields_autoplaced yes)
-		(property "Reference" "H2"
+		(property "Reference" "H3"
 			(at 233.68 38.0999 0)
 			(effects
@@
 			(project "ECE477-SeniorDesign"
 				(path "/527ae649-08be-4368-9cf9-441ebba18eca"
-					(reference "H2")
+					(reference "H3")
 					(unit 1)
 				)
@@
 		(dnp no)
 		(fields_autoplaced yes)
-		(property "Reference" "TP11"
+		(property "Reference" "TP8"
 			(at 204.47 127.5079 0)
 			(effects
@@
 			(project "ECE477-SeniorDesign"
 				(path "/527ae649-08be-4368-9cf9-441ebba18eca"
-					(reference "TP11")
+					(reference "TP8")
 					(unit 1)
 				)
@@
 		(dnp no)
 		(fields_autoplaced yes)
-		(property "Reference" "TP8"
+		(property "Reference" "TP4"
 			(at 193.04 119.8879 0)
 			(effects
@@
 			(project "ECE477-SeniorDesign"
 				(path "/527ae649-08be-4368-9cf9-441ebba18eca"
-					(reference "TP8")
+					(reference "TP4")
 					(unit 1)
 				)
@@
 		(dnp no)
 		(fields_autoplaced yes)
-		(property "Reference" "TP6"
+		(property "Reference" "TP3"
 			(at 193.04 114.8079 0)
 			(effects
@@
 			(project ""
 				(path "/527ae649-08be-4368-9cf9-441ebba18eca"
-					(reference "TP6")
+					(reference "TP3")
 					(unit 1)
 				)
@@
 			)
 		)
+		(pin "switch" input
+			(at 158.75 69.85 270)
+			(effects
+				(font
+					(size 1.27 1.27)
+				)
+				(justify left)
+			)
+		)
 		(instances
 			(project "ECE477-SeniorDesign"
@@
 			(effects
 				(font
+					(size 1.27 1.27)
+				)
+				(justify right)
+			)
+		)
+		(pin "switch" input
+			(at 158.75 86.36 90)
+			(effects
+				(font

Commit message: pushing
Parts:
- TP1, TP2, TP3, TP4, TP5, TP6, TP7, TP8: footprint (none) -> TestPoint:TestPoint_Pad_1.0x1.0mm
Changed lines of the file:
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@@
 			)
 		)
-		(property "Footprint" ""
+		(property "Footprint" "TestPoint:TestPoint_Pad_1.0x1.0mm"
 			(at 93.98 76.2 0)
 			(effects
@@
 			)
 		)
-		(property "Footprint" ""
+		(property "Footprint" "TestPoint:TestPoint_Pad_1.0x1.0mm"
 			(at 104.14 73.66 0)
 			(effects
@@
 			)
 		)
-		(property "Footprint" ""
+		(property "Footprint" "TestPoint:TestPoint_Pad_1.0x1.0mm"
 			(at 207.01 121.92 0)
 			(effects
@@
 			)
 		)
-		(property "Footprint" ""
+		(property "Footprint" "TestPoint:TestPoint_Pad_1.0x1.0mm"
 			(at 207.01 127 0)
 			(effects
@@
 			)
 		)
-		(property "Footprint" ""
+		(property "Footprint" "TestPoint:TestPoint_Pad_1.0x1.0mm"
 			(at 195.58 129.54 0)
 			(effects
@@
 			)
 		)
-		(property "Footprint" ""
+		(property "Footprint" "TestPoint:TestPoint_Pad_1.0x1.0mm"
 			(at 207.01 132.08 0)
 			(effects
@@
 			)
 		)
-		(property "Footprint" ""
+		(property "Footprint" "TestPoint:TestPoint_Pad_1.0x1.0mm"
 			(at 195.58 124.46 0)
 			(effects
@@
 			)
 		)
-		(property "Footprint" ""
+		(property "Footprint" "TestPoint:TestPoint_Pad_1.0x1.0mm"
 			(at 195.58 119.38 0)
 			(effects

Commit message: done
Parts:
- EinkDispCon1: footprint (none) -> Connector_PinHeader_1.00mm:PinHeader_1x08_P1.00mm_Vertical
Changed lines of the file:
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@@
 			)
 		)
-		(property "Footprint" ""
+		(property "Footprint" "Connector_PinHeader_1.00mm:PinHeader_1x08_P1.00mm_Vertical"
 			(at 236.22 120.65 0)
 			(effects

Commit message: push
Parts:
- removed TP1: UART_TX, TestPoint:TestPoint_Pad_1.0x1.0mm, symbol Connector:TestPoint
- removed TP2: UART_RX, TestPoint:TestPoint_Pad_1.0x1.0mm, symbol Connector:TestPoint
- removed TP3: E_MOSI, TestPoint:TestPoint_Pad_1.0x1.0mm, symbol Connector:TestPoint
- removed TP4: E_NSS, TestPoint:TestPoint_Pad_1.0x1.0mm, symbol Connector:TestPoint
- removed TP5: E_RST, TestPoint:TestPoint_Pad_1.0x1.0mm, symbol Connector:TestPoint
- removed TP6: E_SCK, TestPoint:TestPoint_Pad_1.0x1.0mm, symbol Connector:TestPoint
- removed TP7: E_D/C, TestPoint:TestPoint_Pad_1.0x1.0mm, symbol Connector:TestPoint
- removed TP8: E_Busy, TestPoint:TestPoint_Pad_1.0x1.0mm, symbol Connector:TestPoint
Connections:
- net +3.3V: now also EinkDispCon1.8 (BUSY); no longer EinkDispCon1.1 (VCC)
- net GND: now also EinkDispCon1.7 (RST); no longer EinkDispCon1.2 (GND)
- net MCU/Eink_Busy: now also EinkDispCon1.3 (DIN); no longer EinkDispCon1.8 (BUSY)
- net MCU/Eink_D/C: now also EinkDispCon1.5 (CS); no longer EinkDispCon1.6 (D/C)
- net MCU/Eink_RST: now also EinkDispCon1.6 (D/C); no longer EinkDispCon1.7 (RST)
- net MCU/SPI1_MOSI: now also EinkDispCon1.4 (CLK); no longer EinkDispCon1.3 (DIN)
- net MCU/SPI1_NSS: now also EinkDispCon1.1 (VCC); no longer EinkDispCon1.5 (CS)
- net MCU/SPI1_SCK: now also EinkDispCon1.2 (GND); no longer EinkDispCon1.4 (CLK)
Other:
- moved on the sheet: EinkDispCon1

Commit message: push
Parts:
- added TP1, TP2, TP3, TP4, TP5, TP6: TestPoint, TestPoint:TestPoint_Pad_D2.0mm, symbol Connector:TestPoint
- EinkDispCon1: footprint Connector_PinHeader_1.00mm:PinHeader_1x08_P1.00mm_Vertical -> Connector_PinHeader_2.54mm:PinHeader_1x08_P2.54mm_Vertical
Connections:
- net MCU/Eink_Busy: now also TP6.1
- net MCU/Eink_D/C: now also TP4.1
- net MCU/Eink_RST: now also TP5.1
- net MCU/SPI1_MOSI: now also TP1.1
- net MCU/SPI1_NSS: now also TP3.1
- net MCU/SPI1_SCK: now also TP2.1
