File: EInkDisplay-PCB/ECE477-SeniorDesign/ExtraPeriphs_Module_Sheet.kicad_sch (KiCad schematic)
At the start: 24 parts, among them J3 JST Conn, J4 JST Conn, J5 JST Conn, J9 Micro_SD_Card_Det1, U9 74LVC125APW_118

Commit message: whole lotta changes
Parts:
- D1, D2, D3: footprint (none) -> Diode_SMD:D_0805_2012Metric_Pad1.15x1.40mm_HandSolder
- R26, R27, R28: footprint (none) -> Resistor_SMD:R_0805_2012Metric_Pad1.20x1.40mm_HandSolder
- Rr1: renamed from R25; footprint (none) -> Resistor_SMD:R_0805_2012Metric_Pad1.20x1.40mm_HandSolder
Changed lines of the file:
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@@
 	)
 	(junction
-		(at 77.47 172.72)
+		(at 77.47 130.81)
 		(diameter 0)
 		(color 0 0 0 0)
 	)
 	(junction
-		(at 40.64 33.02)
+		(at 77.47 172.72)
 		(diameter 0)
 		(color 0 0 0 0)
 	)
 	(junction
-		(at 64.77 130.81)
+		(at 40.64 33.02)
 		(diameter 0)
 		(color 0 0 0 0)
 	)
 	(junction
-		(at 77.47 130.81)
+		(at 64.77 130.81)
 		(diameter 0)
 		(color 0 0 0 0)
@@
 	(wire
 		(pts
+			(xy 77.47 130.81) (xy 77.47 133.35)
+		)
+		(stroke
+			(width 0)
+			(type default)
+		)
+	)
+	(wire
+		(pts
 			(xy 77.47 186.69) (xy 77.47 181.61)
 		)
@@
 	)
 	(symbol
+		(lib_id "power:GND")
+		(at 77.47 133.35 0)
+		(unit 1)
+		(exclude_from_sim no)
+		(in_bom yes)
+		(on_board yes)
+		(dnp no)
+		(fields_autoplaced yes)
+		(property "Reference" "#PWR014"
+			(at 77.47 139.7 0)
+			(effects
+				(font
+					(size 1.27 1.27)
+				)
+				(hide yes)
+			)
+		)
+		(property "Value" "GND"
+			(at 77.47 138.43 0)
+			(effects
+				(font
+					(size 1.27 1.27)
+				)
+			)
+		)
+		(property "Footprint" ""
+			(at 77.47 133.35 0)
+			(effects
+				(font
+					(size 1.27 1.27)
+				)
+				(hide yes)
+			)
+		)
+		(property "Datasheet" ""
+			(at 77.47 133.35 0)
+			(effects
+				(font
+					(size 1.27 1.27)
+				)
+				(hide yes)
+			)
+		)
+		(property "Description" "Power symbol creates a global label with name \"GND\" , ground"
+			(at 77.47 133.35 0)
+			(effects
+				(font
+					(size 1.27 1.27)
+				)
+				(hide yes)
+			)
+		)
+		(pin "1"
+		)
+		(instances
+			(project "ECE477-SeniorDesign"
+				(path "/527ae649-08be-4368-9cf9-441ebba18eca/9aa04ce4-4558-41ab-8351-e46b80335092"
+					(reference "#PWR014")
+					(unit 1)
+				)
+			)
+		)
+	)
+	(symbol
 		(lib_id "Connector_Generic:Conn_01x02")
 		(at 44.45 139.7 90)
@@
 			)
 		)
-		(property "Footprint" ""
+		(property "Footprint" "Diode_SMD:D_0805_2012Metric_Pad1.15x1.40mm_HandSolder"
 			(at 59.69 172.72 0)
 			(effects
@@
 			)
 		)
-		(property "Footprint" ""
+		(property "Footprint" "Resistor_SMD:R_0805_2012Metric_Pad1.20x1.40mm_HandSolder"
 			(at 33.02 35.56 0)
 			(effects
@@
 			)
 		)
-		(property "Footprint" ""
+		(property "Footprint" "Diode_SMD:D_0805_2012Metric_Pad1.15x1.40mm_HandSolder"
 			(at 59.69 116.84 0)
 			(effects
@@
 	(symbol
 		(lib_id "power:GND")
-		(at 77.47 130.81 0)
-		(unit 1)
-		(exclude_from_sim no)
-		(in_bom yes)
-		(on_board yes)
-		(dnp no)
-		(fields_autoplaced yes)
-		(property "Reference" "#PWR018"
-			(at 77.47 137.16 0)
-			(effects
-				(font
-					(size 1.27 1.27)
-				)
-				(hide yes)
-			)
-		)
-		(property "Value" "GND"
-			(at 77.47 135.89 0)
-			(effects
-				(font
-					(size 1.27 1.27)
-				)
-			)
-		)
-		(property "Footprint" ""
-			(at 77.47 130.81 0)
-			(effects
-				(font
-					(size 1.27 1.27)
-				)
-				(hide yes)
-			)
-		)
-		(property "Datasheet" ""
-			(at 77.47 130.81 0)
-			(effects
-				(font
-					(size 1.27 1.27)
-				)
-				(hide yes)
-			)
-		)
-		(property "Description" "Power symbol creates a global label with name \"GND\" , ground"
-			(at 77.47 130.81 0)
-			(effects
-				(font
-					(size 1.27 1.27)
-				)
-				(hide yes)
-			)
-		)
-		(pin "1"
-		)
-		(instances
-			(project ""
-				(path "/527ae649-08be-4368-9cf9-441ebba18eca/9aa04ce4-4558-41ab-8351-e46b80335092"
-					(reference "#PWR018")
-					(unit 1)
-				)
-			)
-		)
-	)
-	(symbol
-		(lib_id "power:GND")
 		(at 29.21 80.01 270)
 		(unit 1)
@@
 		(dnp no)
 		(fields_autoplaced yes)
-		(property "Reference" "R25"
+		(property "Reference" "Rr1"
 			(at 33.02 22.86 90)
 			(effects
@@
 			)
 		)
-		(property "Footprint" ""
+		(property "Footprint" "Resistor_SMD:R_0805_2012Metric_Pad1.20x1.40mm_HandSolder"
 			(at 33.02 27.94 0)
 			(effects
@@
 			(project ""
 				(path "/527ae649-08be-4368-9cf9-441ebba18eca/9aa04ce4-4558-41ab-8351-e46b80335092"
-					(reference "R25")
+					(reference "Rr1")
 					(unit 1)
 				)
@@
 			)
 		)
-		(property "Footprint" ""
+		(property "Footprint" "Resistor_SMD:R_0805_2012Metric_Pad1.20x1.40mm_HandSolder"
 			(at 93.98 38.1 0)
 			(effects
@@
 			)
 		)
-		(property "Footprint" ""
+		(property "Footprint" "Resistor_SMD:R_0805_2012Metric_Pad1.20x1.40mm_HandSolder"
 			(at 93.98 30.48 0)
 			(effects
@@
 			)
 		)
-		(property "Footprint" ""
+		(property "Footprint" "Diode_SMD:D_0805_2012Metric_Pad1.15x1.40mm_HandSolder"
 			(at 59.69 144.78 0)
 			(effects

Commit message: pushing
Parts:
- removed D1, D2, D3: D, Diode_SMD:D_0805_2012Metric_Pad1.15x1.40mm_HandSolder, symbol Device:D
- added C38: 10pF, Capacitor_SMD:C_0805_2012Metric_Pad1.18x1.45mm_HandSolder, symbol Device:C_Small
- added C39: 100n, Capacitor_SMD:C_0805_2012Metric_Pad1.18x1.45mm_HandSolder, symbol Device:C_Small
- added D1, D2, D3, D4: 1N4148, Diode_THT:D_DO-35_SOD27_P7.62mm_Horizontal, symbol Diode:1N4148
- added J9: JST Conn, PCB_Lib:JST Conn, symbol Connector_Generic:Conn_01x02
- added R20: 100k, Resistor_SMD:R_0805_2012Metric_Pad1.20x1.40mm_HandSolder, symbol Device:R_Small
- added R21: 1k, Resistor_SMD:R_0805_2012Metric_Pad1.20x1.40mm_HandSolder, symbol Device:R_Small
- renumbered C22 to C32, C24 to C33, C26 to C34, C23 to C35, C25 to C36, C27 to C37, J3 to J5, J4 to J6, J5 to J7, J9 to J8, R26 to R11, R10 to R12, R12 to R13, R11 to R15, R13 to R16, R15 to R17, R27 to R18, R28 to R19, U9 to U8
Connections:
- net +3.3V: now also J9.1 (Pin_1)
- net GND: now also C38.2, C39.2, R20.2
- net at J6.2 (Pin_2), R13.1: now also D2.2 (A)
- net at C34.1, R17.1: now also D3.1 (K)
- net at J7.2 (Pin_2), R14.1: now also D3.2 (A)
- net at C33.1, R16.1: now also D2.1 (K)
- net at C32.1, R15.1: now also D1.1 (K)
- net at J5.2 (Pin_2), R12.1: now also D1.2 (A)
- new net: C38.1, D4.1 (K), R21.1
- new net: D4.2 (A), J9.2 (Pin_2), R20.1
- new net switch: C39.1, R21.2

Commit message: pushing
Parts:
- added C40: C_Small, Capacitor_SMD:C_0805_2012Metric_Pad1.18x1.45mm_HandSolder, symbol Device:C_Small
Connections:
- net +3.3V: now also C40.2
- net GND: now also C40.1
Changed lines of the file:
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@@
 	)
 	(junction
+		(at 85.09 25.4)
+		(diameter 0)
+		(color 0 0 0 0)
+	)
+	(junction
 		(at 77.47 144.78)
 		(diameter 0)
@@
 	(wire
 		(pts
-			(xy 85.09 25.4) (xy 88.9 25.4)
+			(xy 85.09 25.4) (xy 99.06 25.4)
 		)
 		(stroke
@@
 	(wire
 		(pts
-			(xy 88.9 25.4) (xy 88.9 22.86)
+			(xy 99.06 25.4) (xy 99.06 22.86)
 		)
 		(stroke
@@
 	)
 	(symbol
+		(lib_id "power:GND")
+		(at 85.09 20.32 180)
+		(unit 1)
+		(exclude_from_sim no)
+		(in_bom yes)
+		(on_board yes)
+		(dnp no)
+		(fields_autoplaced yes)
+		(property "Reference" "#PWR044"
+			(at 85.09 13.97 0)
+			(effects
+				(font
+					(size 1.27 1.27)
+				)
+				(hide yes)
+			)
+		)
+		(property "Value" "GND"
+			(at 85.09 15.24 0)
+			(effects
+				(font
+					(size 1.27 1.27)
+				)
+			)
+		)
+		(property "Footprint" ""
+			(at 85.09 20.32 0)
+			(effects
+				(font
+					(size 1.27 1.27)
+				)
+				(hide yes)
+			)
+		)
+		(property "Datasheet" ""
+			(at 85.09 20.32 0)
+			(effects
+				(font
+					(size 1.27 1.27)
+				)
+				(hide yes)
+			)
+		)
+		(property "Description" "Power symbol creates a global label with name \"GND\" , ground"
+			(at 85.09 20.32 0)
+			(effects
+				(font
+					(size 1.27 1.27)
+				)
+				(hide yes)
+			)
+		)
+		(pin "1"
+		)
+		(instances
+			(project ""
+				(path "/527ae649-08be-4368-9cf9-441ebba18eca/9aa04ce4-4558-41ab-8351-e46b80335092"
+					(reference "#PWR044")
+					(unit 1)
+				)
+			)
+		)
+	)
+	(symbol
 		(lib_id "Device:R_Small")
 		(at 54.61 179.07 0)
@@
 	(symbol
 		(lib_id "power:+3.3V")
-		(at 88.9 22.86 0)
+		(at 99.06 22.86 0)
 		(unit 1)
 		(exclude_from_sim no)
@@
 		(fields_autoplaced yes)
 		(property "Reference" "#PWR039"
-			(at 88.9 26.67 0)
+			(at 99.06 26.67 0)
 			(effects
 				(font
@@
 		)
 		(property "Value" "+3.3V"
-			(at 88.9 17.78 0)
+			(at 99.06 17.78 0)
 			(effects
 				(font
@@
 		)
 		(property "Footprint" ""
-			(at 88.9 22.86 0)
+			(at 99.06 22.86 0)
 			(effects
 				(font
@@
 		)
 		(property "Datasheet" ""
-			(at 88.9 22.86 0)
+			(at 99.06 22.86 0)
 			(effects
 				(font
@@
 		)
 		(property "Description" "Power symbol creates a global label with name \"+3.3V\""
-			(at 88.9 22.86 0)
+			(at 99.06 22.86 0)
 			(effects
 				(font
@@
 					(unit 1)
 				)
+			)
+		)
+	)
+	(symbol
+		(lib_id "Device:C_Small")
+		(at 85.09 22.86 0)
+		(unit 1)
+		(exclude_from_sim no)
+		(in_bom yes)
+		(on_board yes)
+		(dnp no)
+		(fields_autoplaced yes)
+		(property "Reference" "C40"
+			(at 87.63 21.5962 0)
+			(effects
+				(font
+					(size 1.27 1.27)
+				)
+				(justify left)
+			)
+		)
+		(property "Value" "C_Small"
+			(at 87.63 24.1362 0)
+			(effects
+				(font
+					(size 1.27 1.27)
+				)
+				(justify left)
+			)
+		)
+		(property "Footprint" "Capacitor_SMD:C_0805_2012Metric_Pad1.18x1.45mm_HandSolder"
+			(at 85.09 22.86 0)
+			(effects
+				(font
+					(size 1.27 1.27)
+				)
+				(hide yes)
+			)
+		)
+		(property "Datasheet" "~"
+			(at 85.09 22.86 0)
+			(effects
+				(font
+					(size 1.27 1.27)
+				)
+				(hide yes)
+			)
+		)
+		(property "Description" "Unpolarized capacitor, small symbol"
+			(at 85.09 22.86 0)
+			(effects
+				(font
+					(size 1.27 1.27)
+				)
+				(hide yes)
+			)
+		)
+		(pin "2"
+		)
+		(pin "1"
+		)
+		(instances
+			(project ""
+				(path "/527ae649-08be-4368-9cf9-441ebba18eca/9aa04ce4-4558-41ab-8351-e46b80335092"
+					(reference "C40")
+					(unit 1)
+				)

Commit message: pushing
Parts:
- renumbered C32 to C35, C33 to C36, C34 to C37, C35 to C38, C36 to C39, C37 to C40, C40 to C41, C38 to C42, C39 to C43, D1 to D4, D2 to D5, D3 to D6, D4 to D7, J7 to J10, J8 to J11, J9 to J12, J5 to J8, J6 to J9, R11 to R19, R12 to R20, R13 to R21, R14 to R22, R15 to R23, R16 to R24, R17 to R25, R18 to R26, R19 to R27, R20 to R28, R21 to R29, U8 to U9

Commit message: push
Parts:
- removed J11: Micro_SD_Card_Det1, PCB_Lib:SD_Reader, symbol Connector:Micro_SD_Card_Det1
- added CARD1: ~, PCB_Lib:SD_reader_comp, symbol EinkComponentLibrary:XKTF-015-N
Connections:
- net CS_LLC is gone; now on net CS_LLS: U9.8 (3Y)
- net DO_LLC is gone; now on net DO_LLS: R26.2
- net +3.3V: now also CARD1.4 (VDD)
- net CS_LLS: now also CARD1.2 (CD/DAT3)
- net DI_LLS: now also CARD1.3 (CMD)
- net DO_LLS: now also CARD1.7 (DAT0)
- net GND: now also CARD1.10 (GND), CARD1.11 (GND), CARD1.12 (GND), CARD1.13 (GND), CARD1.6 (VSS)
- net SCK_LLS: now also CARD1.5 (CLK)
- no-connect marks 4 -> 3

Commit message: push
Parts:
- removed J8: JST Conn, PCB_Lib:JST Conn, symbol Connector_Generic:Conn_01x02
- added J5: Conn_01x02, Connector_Wire:SolderWire-0.1sqmm_1x02_P3.6mm_D0.4mm_OD1mm, symbol Connector_Generic:Conn_01x02
- J10, J12, J9: footprint PCB_Lib:JST Conn -> Connector_Wire:SolderWire-0.1sqmm_1x02_P3.6mm_D0.4mm_OD1mm
Connections:
- net +3.3V: now also J5.1 (Pin_1)
- net at D4.2 (A), R20.1: now also J5.2 (Pin_2)
Changed lines of the file:
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@@
 			)
 		)
-		(property "Footprint" "PCB_Lib:JST Conn"
+		(property "Footprint" "Connector_Wire:SolderWire-0.1sqmm_1x02_P3.6mm_D0.4mm_OD1mm"
 			(at 44.45 139.7 0)
 			(effects
@@
 	)
 	(symbol
+		(lib_id "Connector_Generic:Conn_01x02")
+		(at 44.45 111.76 90)
+		(unit 1)
+		(exclude_from_sim no)
+		(in_bom yes)
+		(on_board yes)
+		(dnp no)
+		(fields_autoplaced yes)
+		(property "Reference" "J5"
+			(at 49.53 110.4899 90)
+			(effects
+				(font
+					(size 1.27 1.27)
+				)
+				(justify right)
+			)
+		)
+		(property "Value" "Conn_01x02"
+			(at 49.53 113.0299 90)
+			(effects
+				(font
+					(size 1.27 1.27)
+				)
+				(justify right)
+			)
+		)
+		(property "Footprint" "Connector_Wire:SolderWire-0.1sqmm_1x02_P3.6mm_D0.4mm_OD1mm"
+			(at 44.45 111.76 0)
+			(effects
+				(font
+					(size 1.27 1.27)
+				)
+				(hide yes)
+			)
+		)
+		(property "Datasheet" "~"
+			(at 44.45 111.76 0)
+			(effects
+				(font
+					(size 1.27 1.27)
+				)
+				(hide yes)
+			)
+		)
+		(property "Description" "Generic connector, single row, 01x02, script generated (kicad-library-utils/schlib/autogen/connector/)"
+			(at 44.45 111.76 0)
+			(effects
+				(font
+					(size 1.27 1.27)
+				)
+				(hide yes)
+			)
+		)
+		(pin "1"
+		)
+		(pin "2"
+		)
+		(instances
+			(project ""
+				(path "/527ae649-08be-4368-9cf9-441ebba18eca/9aa04ce4-4558-41ab-8351-e46b80335092"
+					(reference "J5")
+					(unit 1)
+				)
+			)
+		)
+	)
+	(symbol
 		(lib_id "Device:R_Small")
 		(at 54.61 151.13 0)
@@
 			)
 		)
-		(property "Footprint" "PCB_Lib:JST Conn"
+		(property "Footprint" "Connector_Wire:SolderWire-0.1sqmm_1x02_P3.6mm_D0.4mm_OD1mm"
 			(at 44.45 167.64 0)
 			(effects
@@
 	)
 	(symbol
-		(lib_id "Connector_Generic:Conn_01x02")
-		(at 44.45 111.76 90)
-		(unit 1)
-		(exclude_from_sim no)
-		(in_bom yes)
-		(on_board yes)
-		(dnp no)
-		(fields_autoplaced yes)
-		(property "Reference" "J8"
-			(at 49.53 110.4899 90)
-			(effects
-				(font
-					(size 1.27 1.27)
-				)
-				(justify right)
-			)
-		)
-		(property "Value" "JST Conn"
-			(at 49.53 113.0299 90)
-			(effects
-				(font
-					(size 1.27 1.27)
-				)
-				(justify right)
-			)
-		)
-		(property "Footprint" "PCB_Lib:JST Conn"
-			(at 44.45 111.76 0)
-			(effects
-				(font
-					(size 1.27 1.27)
-				)
-				(hide yes)
-			)
-		)
-		(property "Datasheet" "~"
-			(at 44.45 111.76 0)
-			(effects
-				(font
-					(size 1.27 1.27)
-				)
-				(hide yes)
-			)
-		)
-		(property "Description" "Generic connector, single row, 01x02, script generated (kicad-library-utils/schlib/autogen/connector/)"
-			(at 44.45 111.76 0)
-			(effects
-				(font
-					(size 1.27 1.27)
-				)
-				(hide yes)
-			)
-		)
-		(pin "1"
-		)
-		(pin "2"
-		)
-		(instances
-			(project ""
-				(path "/527ae649-08be-4368-9cf9-441ebba18eca/9aa04ce4-4558-41ab-8351-e46b80335092"
-					(reference "J8")
-					(unit 1)
-				)
-			)
-		)
-	)
-	(symbol
 		(lib_id "Device:R_Small")
 		(at 72.39 116.84 90)
@@
 			)
 		)
-		(property "Footprint" "PCB_Lib:JST Conn"
+		(property "Footprint" "Connector_Wire:SolderWire-0.1sqmm_1x02_P3.6mm_D0.4mm_OD1mm"
 			(at 115.57 144.78 0)
 			(effects
