File: EInkDisplay-PCB/ECE477-SeniorDesign/MCU_Module_Sheet.kicad_sch (KiCad schematic)
At the start: 42 parts, among them J2 Conn_01x05_Pin, J7 Conn_01x05, U3 STM32L496ZGTxP, U7 PTS526 SK15 SMTR2 LFS, Y1 Y1

Commit message: pushing
Parts:
- added TP18: ~, symbol Connector:TestPoint
- renumbered C28 to C1, C18 to C16, C16 to C18, C29 to C2, C20 to C3, C19 to C4, C1 to C5, C2 to C6, C3 to C7, C4 to C8, J7 to J1, SWBOOT0 to SWBOOT1, TP18 to TP10, TP19 to TP11, TP20 to TP12, TP15 to TP13, TP16 to TP14, TP25 to TP15, TP27 to TP16, TP29 to TP17, TP26 to TP19, TP28 to TP20, TP31 to TP21, TP30 to TP22, TP32 to TP23, TP21 to TP24, TP23 to TP25, TP22 to TP26, TP17 to TP9, U7 to U1, U3 to U2
Connections:
- net switch: now reaches U2.4 (PE5)
- net switch: now also TP18.1
- no-connect marks 78 -> 77

Commit message: pushing
Parts:
- added J10, J11: Conn_01x05_Pin, Connector_PinHeader_1.00mm:PinHeader_1x05_P1.00mm_Vertical, symbol Connector:Conn_01x05_Pin
- SWBOOT1: footprint PCB_Lib:PCM12SMTR_CNK -> Button_Switch_SMD:SW_SPDT_PCM12
- TP10, TP11, TP12, TP13, TP14, TP15, TP16, TP17, TP18, TP19, TP20, TP21, TP22, TP23, TP24, TP25, TP26, TP9: footprint (none) -> TestPoint:TestPoint_Pad_1.0x1.0mm
Connections:
- net Extra_3: no longer TP23.1, U2.45 (PC5)
- net Extra_4: no longer TP21.1, U2.44 (PC4)
- net Extra_5: no longer TP22.1, U2.29 (PC3)
- net GPIO_3: now also TP24.1
- net GPIO_4: now also TP23.1
- net GPIO_5: now also TP22.1
- net GPIO_6: now also TP21.1
- net I2C2_SDA: now also TP26.1
- net I2C4_SCL: now also J11.4 (Pin_4)
- net I2C4_SDA: now also J11.5 (Pin_5)
- net SPI2_MISO: now also J10.4 (Pin_4)
- net SPI2_MOSI: now also J10.3 (Pin_3)
- net SPI2_NSS: now also J10.2 (Pin_2)
- net SPI2_SCK: now also J10.5 (Pin_5)
- net USART2_RX: now also J11.2 (Pin_2); no longer TP26.1
- net USART2_TX: now also J11.3 (Pin_3); no longer TP24.1
- no-connect marks 77 -> 82
Other:
- note added: "Extra UART and I2C"
- moved on the sheet: J1, J2

Commit message: pushing
Parts:
- added R22: R_Small, Resistor_SMD:R_0805_2012Metric_Pad1.20x1.40mm_HandSolder, symbol Device:R_Small
Connections:
- net +3.3V: now also R22.2
- net NRST: now also R22.1
Other:
- moved on the sheet: C3, TP13

Commit message: pushing
Parts:
- renumbered C3 to C1, C1 to C2, C2 to C3, J10 to J3, J11 to J4, R22 to R1, R1 to R2, TP9 to TP10, TP10 to TP11, TP11 to TP12, TP12 to TP13, TP25 to TP21, TP21 to TP22, TP22 to TP23, TP23 to TP24, TP24 to TP25, TP13 to TP9
Changed lines of the file:
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@@
 		(on_board yes)
 		(dnp no)
-		(property "Reference" "TP25"
+		(property "Reference" "TP21"
 			(at 243.078 208.534 90)
 			(effects
@@
 			(project "ECE477-SeniorDesign"
 				(path "/527ae649-08be-4368-9cf9-441ebba18eca/a47b6934-98dd-4056-b1df-1ab751d1c2a0"
-					(reference "TP25")
+					(reference "TP21")
 					(unit 1)
 				)
@@
 		(on_board yes)
 		(dnp no)
-		(property "Reference" "TP22"
+		(property "Reference" "TP23"
 			(at 255.778 200.914 90)
 			(effects
@@
 			(project "ECE477-SeniorDesign"
 				(path "/527ae649-08be-4368-9cf9-441ebba18eca/a47b6934-98dd-4056-b1df-1ab751d1c2a0"
-					(reference "TP22")
+					(reference "TP23")
 					(unit 1)
 				)
@@
 		(dnp no)
 		(fields_autoplaced yes)
-		(property "Reference" "J10"
+		(property "Reference" "J3"
 			(at 60.96 91.4399 0)
 			(effects
@@
 			(project "ECE477-SeniorDesign"
 				(path "/527ae649-08be-4368-9cf9-441ebba18eca/a47b6934-98dd-4056-b1df-1ab751d1c2a0"
-					(reference "J10")
+					(reference "J3")
 					(unit 1)
 				)
@@
 		(on_board yes)
 		(dnp no)
-		(property "Reference" "TP23"
+		(property "Reference" "TP24"
 			(at 260.858 203.454 90)
 			(effects
@@
 			(project "ECE477-SeniorDesign"
 				(path "/527ae649-08be-4368-9cf9-441ebba18eca/a47b6934-98dd-4056-b1df-1ab751d1c2a0"
-					(reference "TP23")
+					(reference "TP24")
 					(unit 1)
 				)
@@
 		(dnp no)
 		(fields_autoplaced yes)
-		(property "Reference" "R1"
+		(property "Reference" "R2"
 			(at 152.4 81.28 90)
 			(effects
@@
 			(project ""
 				(path "/527ae649-08be-4368-9cf9-441ebba18eca/a47b6934-98dd-4056-b1df-1ab751d1c2a0"
-					(reference "R1")
+					(reference "R2")
 					(unit 1)
 				)
@@
 		(on_board yes)
 		(dnp no)
-		(property "Reference" "C3"
+		(property "Reference" "C1"
 			(at 117.348 46.228 0)
 			(effects
@@
 			(project ""
 				(path "/527ae649-08be-4368-9cf9-441ebba18eca/a47b6934-98dd-4056-b1df-1ab751d1c2a0"
-					(reference "C3")
+					(reference "C1")
 					(unit 1)
 				)
@@
 		(dnp no)
 		(fields_autoplaced yes)
-		(property "Reference" "J11"
+		(property "Reference" "J4"
 			(at 60.96 116.8399 0)
 			(effects
@@
 			(project "ECE477-SeniorDesign"
 				(path "/527ae649-08be-4368-9cf9-441ebba18eca/a47b6934-98dd-4056-b1df-1ab751d1c2a0"
-					(reference "J11")
+					(reference "J4")
 					(unit 1)
 				)
@@
 		(on_board yes)
 		(dnp no)
-		(property "Reference" "TP24"
+		(property "Reference" "TP25"
 			(at 265.938 205.994 90)
 			(effects
@@
 			(project "ECE477-SeniorDesign"
 				(path "/527ae649-08be-4368-9cf9-441ebba18eca/a47b6934-98dd-4056-b1df-1ab751d1c2a0"
-					(reference "TP24")
+					(reference "TP25")
 					(unit 1)
 				)
@@
 		(dnp no)
 		(fields_autoplaced yes)
-		(property "Reference" "#PWR05"
+		(property "Reference" "#PWR07"
 			(at 134.62 17.78 0)
 			(effects
@@
 			(project "ECE477-SeniorDesign"
 				(path "/527ae649-08be-4368-9cf9-441ebba18eca/a47b6934-98dd-4056-b1df-1ab751d1c2a0"
-					(reference "#PWR05")
+					(reference "#PWR07")
 					(unit 1)
 				)
@@
 		(dnp no)
 		(fields_autoplaced yes)
-		(property "Reference" "#PWR07"
+		(property "Reference" "#PWR09"
 			(at 158.75 68.58 0)
 			(effects
@@
 			(project ""
 				(path "/527ae649-08be-4368-9cf9-441ebba18eca/a47b6934-98dd-4056-b1df-1ab751d1c2a0"
-					(reference "#PWR07")
+					(reference "#PWR09")
 					(unit 1)
 				)
@@
 		(dnp no)
 		(fields_autoplaced yes)
-		(property "Reference" "#PWR043"
+		(property "Reference" "#PWR04"
 			(at 121.92 60.96 0)
 			(effects
@@
 			(project ""
 				(path "/527ae649-08be-4368-9cf9-441ebba18eca/a47b6934-98dd-4056-b1df-1ab751d1c2a0"
-					(reference "#PWR043")
+					(reference "#PWR04")
 					(unit 1)
 				)
@@
 		(on_board yes)
 		(dnp no)
-		(property "Reference" "TP12"
+		(property "Reference" "TP13"
 			(at 126.746 119.888 90)
 			(effects
@@
 			(project "ECE477-SeniorDesign"
 				(path "/527ae649-08be-4368-9cf9-441ebba18eca/a47b6934-98dd-4056-b1df-1ab751d1c2a0"
-					(reference "TP12")
+					(reference "TP13")
 					(unit 1)
 				)
@@
 		(dnp no)
 		(fields_autoplaced yes)
-		(property "Reference" "#PWR03"
+		(property "Reference" "#PWR05"
 			(at 128.27 86.36 0)
 			(effects
@@
 			(project ""
 				(path "/527ae649-08be-4368-9cf9-441ebba18eca/a47b6934-98dd-4056-b1df-1ab751d1c2a0"
-					(reference "#PWR03")
+					(reference "#PWR05")
 					(unit 1)
 				)
@@
 		(dnp no)
 		(fields_autoplaced yes)
-		(property "Reference" "R22"
+		(property "Reference" "R1"
 			(at 124.46 58.4199 0)
 			(effects
@@
 			(project ""
 				(path "/527ae649-08be-4368-9cf9-441ebba18eca/a47b6934-98dd-4056-b1df-1ab751d1c2a0"
-					(reference "R22")
+					(reference "R1")
 					(unit 1)
 				)
@@
 		(dnp no)
 		(fields_autoplaced yes)
-		(property "Reference" "#PWR09"
+		(property "Reference" "#PWR010"
 			(at 175.26 31.75 0)
 			(effects
@@
 			(project ""
 				(path "/527ae649-08be-4368-9cf9-441ebba18eca/a47b6934-98dd-4056-b1df-1ab751d1c2a0"
-					(reference "#PWR09")
+					(reference "#PWR010")
 					(unit 1)
 				)
@@
 		(on_board yes)
 		(dnp no)
-		(property "Reference" "TP10"
+		(property "Reference" "TP11"
 			(at 117.094 107.442 90)
 			(effects
@@
 			(project "ECE477-SeniorDesign"
 				(path "/527ae649-08be-4368-9cf9-441ebba18eca/a47b6934-98dd-4056-b1df-1ab751d1c2a0"
-					(reference "TP10")
+					(reference "TP11")
 					(unit 1)
 				)
@@
 		(on_board yes)
 		(dnp no)
-		(property "Reference" "#PWR06"
+		(property "Reference" "#PWR08"
 			(at 140.97 78.74 0)
 			(effects
@@
 			(project ""
 				(path "/527ae649-08be-4368-9cf9-441ebba18eca/a47b6934-98dd-4056-b1df-1ab751d1c2a0"
-					(reference "#PWR06")
+					(reference "#PWR08")
 					(unit 1)
 				)
@@
 		(on_board yes)
 		(dnp no)
-		(property "Reference" "TP13"
+		(property "Reference" "TP9"
 			(at 103.632 56.388 0)
 			(effects
@@
 			(project ""
 				(path "/527ae649-08be-4368-9cf9-441ebba18eca/a47b6934-98dd-4056-b1df-1ab751d1c2a0"
-					(reference "TP13")
+					(reference "TP9")
 					(unit 1)
 				)
@@
 		(on_board yes)
 		(dnp no)
-		(property "Reference" "TP11"
+		(property "Reference" "TP12"
 			(at 125.476 113.538 90)
 			(effects
@@
 			(project "ECE477-SeniorDesign"
 				(path "/527ae649-08be-4368-9cf9-441ebba18eca/a47b6934-98dd-4056-b1df-1ab751d1c2a0"
-					(reference "TP11")
+					(reference "TP12")
 					(unit 1)
 				)
@@
 		(on_board yes)
 		(dnp no)
-		(property "Reference" "TP9"
+		(property "Reference" "TP10"
 			(at 115.824 103.632 90)
 			(effects
@@
 			(project "ECE477-SeniorDesign"
 				(path "/527ae649-08be-4368-9cf9-441ebba18eca/a47b6934-98dd-4056-b1df-1ab751d1c2a0"
-					(reference "TP9")
+					(reference "TP10")
 					(unit 1)
 				)
@@
 		(dnp no)
 		(fields_autoplaced yes)
-		(property "Reference" "#PWR011"
+		(property "Reference" "#PWR012"
 			(at 243.84 49.53 0)
 			(effects
@@
 			(project ""
 				(path "/527ae649-08be-4368-9cf9-441ebba18eca/a47b6934-98dd-4056-b1df-1ab751d1c2a0"
-					(reference "#PWR011")
+					(reference "#PWR012")
 					(unit 1)
 				)
@@
 		(on_board yes)
 		(dnp no)
-		(property "Reference" "C2"
+		(property "Reference" "C3"
 			(at 151.892 69.85 0)
 			(effects
@@
 			(project "ECE477-SeniorDesign"
 				(path "/527ae649-08be-4368-9cf9-441ebba18eca/a47b6934-98dd-4056-b1df-1ab751d1c2a0"
-					(reference "C2")
+					(reference "C3")
 					(unit 1)
 				)
@@
 		(dnp no)
 		(fields_autoplaced yes)
-		(property "Reference" "#PWR08"
+		(property "Reference" "#PWR03"
 			(at 121.92 39.37 0)
 			(effects
@@
 			(project ""
 				(path "/527ae649-08be-4368-9cf9-441ebba18eca/a47b6934-98dd-4056-b1df-1ab751d1c2a0"
-					(reference "#PWR08")
+					(reference "#PWR03")
 					(unit 1)
 				)
@@
 		(on_board yes)
 		(dnp no)
-		(property "Reference" "TP21"
+		(property "Reference" "TP22"
 			(at 250.698 198.374 90)
 			(effects
@@
 			(project "ECE477-SeniorDesign"
 				(path "/527ae649-08be-4368-9cf9-441ebba18eca/a47b6934-98dd-4056-b1df-1ab751d1c2a0"
-					(reference "TP21")
+					(reference "TP22")
 					(unit 1)
 				)
@@
 		(dnp no)
 		(fields_autoplaced yes)
-		(property "Reference" "#PWR010"
+		(property "Reference" "#PWR011"
 			(at 200.66 238.76 0)
 			(effects
@@
 			(project ""
 				(path "/527ae649-08be-4368-9cf9-441ebba18eca/a47b6934-98dd-4056-b1df-1ab751d1c2a0"
-					(reference "#PWR010")
+					(reference "#PWR011")
 					(unit 1)
 				)
@@
 		(dnp no)
 		(fields_autoplaced yes)
-		(property "Reference" "#PWR04"
+		(property "Reference" "#PWR06"
 			(at 130.81 99.06 0)
 			(effects
@@
 			(project ""
 				(path "/527ae649-08be-4368-9cf9-441ebba18eca/a47b6934-98dd-4056-b1df-1ab751d1c2a0"
-					(reference "#PWR04")
+					(reference "#PWR06")
 					(unit 1)
 				)
@@
 		(on_board yes)
 		(dnp no)
-		(property "Reference" "C1"
+		(property "Reference" "C2"
 			(at 132.588 68.072 0)
 			(effects
@@
 			(project "ECE477-SeniorDesign"
 				(path "/527ae649-08be-4368-9cf9-441ebba18eca/a47b6934-98dd-4056-b1df-1ab751d1c2a0"
-					(reference "C1")
+					(reference "C2")
 					(unit 1)
 				)

Commit message: push
Parts:
- removed TP10, TP11, TP12, TP13, TP15, TP16, TP17, TP18, TP19, TP20, TP21, TP22, TP23, TP24, TP25, TP26: ~, TestPoint:TestPoint_Pad_1.0x1.0mm, symbol Connector:TestPoint
- removed TP14: BOOT0, TestPoint:TestPoint_Pad_1.0x1.0mm, symbol Connector:TestPoint
- removed TP9: NSRT, TestPoint:TestPoint_Pad_1.0x1.0mm, symbol Connector:TestPoint
Connections:
- net Eink_D/C: now also U2.44 (PC4); no longer U2.103 (PA11)
- net Eink_RST: now also U2.45 (PC5); no longer U2.104 (PA12)

Commit message: push
Parts:
- removed J1: Conn_01x05, symbol Connector_Generic:Conn_01x05
- removed Y1: Y1, PCB_Lib:XTAL_ABS04W-32.768KHZ-4-D2-T5, symbol Device:Crystal_GND24_Small
- added J1: Conn_01x05_Pin, Connector_PinHeader_1.00mm:PinHeader_1x05_P1.00mm_Vertical, symbol Connector:Conn_01x05_Pin
- added Y1: CM9V-T1A-32.768KHZ-7PF-100PPM-TA-QC, PCB_Lib:CM9V-T1A-32.768KHZ-7PF-100PPM-TA-QC, symbol EinkComponentLibrary:CM9V-T1A-32.768KHZ-7PF-100PPM-TA-QC
- C2: value 4pF -> 6pF
- C3: value 4pF -> 6pf
Connections:
- net +3.3V: now also J1.5 (Pin_5)
- net GND: now also J1.4 (Pin_4)
- net NRST: now also J1.3 (Pin_3)
- net SPI2_MISO: now also U2.117 (PD3); no longer U2.75 (PB14)
- net SPI2_MOSI: now also J3.5 (Pin_5), U2.118 (PD4); no longer J3.3 (Pin_3), U2.76 (PB15)
- net SPI2_NSS: now also U2.114 (PD0); no longer U2.139 (PB9)
- net SPI2_SCK: now also J3.3 (Pin_3), U2.115 (PD1); no longer J3.5 (Pin_5), U2.69 (PB10)
- net SWCLK: now also J1.1 (Pin_1)
- net SWDIO: now also J1.2 (Pin_2)
- net USART2_RX: now also J4.3 (Pin_3); no longer J4.2 (Pin_2)
- net USART2_TX: now also J4.2 (Pin_2); no longer J4.3 (Pin_3)
- net at C2.2, U2.23 (PH0): now also Y1.1
- net at C3.2, U2.24 (PH1): now also Y1.2
- no-connect marks 82 -> 79

Commit message: push
Parts:
- J1, J2, J3, J4: footprint Connector_PinHeader_1.00mm:PinHeader_1x05_P1.00mm_Vertical -> Connector_PinHeader_2.54mm:PinHeader_1x05_P2.54mm_Vertical
Changed lines of the file:
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@@
 			)
 		)
-		(property "Footprint" "Connector_PinHeader_1.00mm:PinHeader_1x05_P1.00mm_Vertical"
+		(property "Footprint" "Connector_PinHeader_2.54mm:PinHeader_1x05_P2.54mm_Vertical"
 			(at 59.69 92.71 0)
 			(effects
@@
 			)
 		)
-		(property "Footprint" "Connector_PinHeader_1.00mm:PinHeader_1x05_P1.00mm_Vertical"
+		(property "Footprint" "Connector_PinHeader_2.54mm:PinHeader_1x05_P2.54mm_Vertical"
 			(at 59.69 118.11 0)
 			(effects
@@
 			)
 		)
-		(property "Footprint" "Connector_PinHeader_1.00mm:PinHeader_1x05_P1.00mm_Vertical"
+		(property "Footprint" "Connector_PinHeader_2.54mm:PinHeader_1x05_P2.54mm_Vertical"
 			(at 59.69 40.64 0)
 			(effects
@@
 			)
 		)
-		(property "Footprint" "Connector_PinHeader_1.00mm:PinHeader_1x05_P1.00mm_Vertical"
+		(property "Footprint" "Connector_PinHeader_2.54mm:PinHeader_1x05_P2.54mm_Vertical"
 			(at 59.69 66.04 0)
 			(effects

Commit message: rev 2
Parts:
- C10, C11, C12, C13, C14, C15, C16, C17, C4, C5, C6, C7, C8, C9: footprint Capacitor_SMD:C_0603_1608Metric_Pad1.08x0.95mm_HandSolder -> Capacitor_SMD:C_0805_2012Metric_Pad1.18x1.45mm_HandSolder
Changed lines of the file:
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@@
 			)
 		)
-		(property "Footprint" "Capacitor_SMD:C_0603_1608Metric_Pad1.08x0.95mm_HandSolder"
+		(property "Footprint" "Capacitor_SMD:C_0805_2012Metric_Pad1.18x1.45mm_HandSolder"
 			(at 195.58 34.29 0)
 			(effects
@@
 			)
 		)
-		(property "Footprint" "Capacitor_SMD:C_0603_1608Metric_Pad1.08x0.95mm_HandSolder"
+		(property "Footprint" "Capacitor_SMD:C_0805_2012Metric_Pad1.18x1.45mm_HandSolder"
 			(at 233.68 34.29 0)
 			(effects
@@
 			)
 		)
-		(property "Footprint" "Capacitor_SMD:C_0603_1608Metric_Pad1.08x0.95mm_HandSolder"
+		(property "Footprint" "Capacitor_SMD:C_0805_2012Metric_Pad1.18x1.45mm_HandSolder"
 			(at 223.52 34.29 0)
 			(effects
@@
 			)
 		)
-		(property "Footprint" "Capacitor_SMD:C_0603_1608Metric_Pad1.08x0.95mm_HandSolder"
+		(property "Footprint" "Capacitor_SMD:C_0805_2012Metric_Pad1.18x1.45mm_HandSolder"
 			(at 179.07 34.29 0)
 			(effects
@@
 			)
 		)
-		(property "Footprint" "Capacitor_SMD:C_0603_1608Metric_Pad1.08x0.95mm_HandSolder"
+		(property "Footprint" "Capacitor_SMD:C_0805_2012Metric_Pad1.18x1.45mm_HandSolder"
 			(at 228.6 34.29 0)
 			(effects
@@
 			)
 		)
-		(property "Footprint" "Capacitor_SMD:C_0603_1608Metric_Pad1.08x0.95mm_HandSolder"
+		(property "Footprint" "Capacitor_SMD:C_0805_2012Metric_Pad1.18x1.45mm_HandSolder"
 			(at 238.76 34.29 0)
 			(effects
@@
 			)
 		)
-		(property "Footprint" "Capacitor_SMD:C_0603_1608Metric_Pad1.08x0.95mm_HandSolder"
+		(property "Footprint" "Capacitor_SMD:C_0805_2012Metric_Pad1.18x1.45mm_HandSolder"
 			(at 187.96 34.29 0)
 			(effects
@@
 			)
 		)
-		(property "Footprint" "Capacitor_SMD:C_0603_1608Metric_Pad1.08x0.95mm_HandSolder"
+		(property "Footprint" "Capacitor_SMD:C_0805_2012Metric_Pad1.18x1.45mm_HandSolder"
 			(at 184.15 34.29 0)
 			(effects
@@
 			)
 		)
-		(property "Footprint" "Capacitor_SMD:C_0603_1608Metric_Pad1.08x0.95mm_HandSolder"
+		(property "Footprint" "Capacitor_SMD:C_0805_2012Metric_Pad1.18x1.45mm_HandSolder"
 			(at 191.77 34.29 0)
 			(effects
@@
 			)
 		)
-		(property "Footprint" "Capacitor_SMD:C_0603_1608Metric_Pad1.08x0.95mm_HandSolder"
+		(property "Footprint" "Capacitor_SMD:C_0805_2012Metric_Pad1.18x1.45mm_HandSolder"
 			(at 203.2 34.29 0)
 			(effects
@@
 			)
 		)
-		(property "Footprint" "Capacitor_SMD:C_0603_1608Metric_Pad1.08x0.95mm_HandSolder"
+		(property "Footprint" "Capacitor_SMD:C_0805_2012Metric_Pad1.18x1.45mm_HandSolder"
 			(at 218.44 34.29 0)
 			(effects
@@
 			)
 		)
-		(property "Footprint" "Capacitor_SMD:C_0603_1608Metric_Pad1.08x0.95mm_HandSolder"
+		(property "Footprint" "Capacitor_SMD:C_0805_2012Metric_Pad1.18x1.45mm_HandSolder"
 			(at 199.39 34.29 0)
 			(effects
@@
 			)
 		)
-		(property "Footprint" "Capacitor_SMD:C_0603_1608Metric_Pad1.08x0.95mm_HandSolder"
+		(property "Footprint" "Capacitor_SMD:C_0805_2012Metric_Pad1.18x1.45mm_HandSolder"
 			(at 213.36 34.29 0)
 			(effects
@@
 			)
 		)
-		(property "Footprint" "Capacitor_SMD:C_0603_1608Metric_Pad1.08x0.95mm_HandSolder"
+		(property "Footprint" "Capacitor_SMD:C_0805_2012Metric_Pad1.18x1.45mm_HandSolder"
 			(at 208.28 34.29 0)
 			(effects
